File: _autosave-PickleRick.kicad_pcb (KiCad board)
At the start: 4 copper layers, 100 x 37 mm, 171 parts, among them J1 RBUS, J10 Conn_Coaxial, J11 Conn_Coaxial, J12 Conn_01x03_Male, J2 Conn_01x02_Male, J3 292227-7, J4 Micro_SD_Card_Det, J5 USB_C_Receptacle_USB2.0, J6 Screw_Terminal_01x08, J7 Conn_01x05_Male, J8 DeployLipo, J9 UCLipo, Q1 PMV20ENR, Q2 NCV8415STT1G, Q3 NCV8415STT1G, Q4 NCV8415STT1G, Q5 NCV8415STT1G, Q6 SI4143DY-T1-GE3, Q7 SI4143DY-T1-GE3, U1 ESP32-S3, U10 NCP1117-3.3_SOT223, U11 XC8111, U12 XC8111, U13 XC8111, U14 LTC4412xS6, U15 MAX77827AEFD+T, U16 SC4215, U17 LTC4412xS6, U18 XC8111, U19 MAX-M10S, U2 DPS310, U20 SN65HVD230, U21 RFM95W-868S2, U3 LTV-247, U4 PCA9534RGVR, U5 PCA9685BS, U6 H3LIS331DLTR, U7 ICM-20608-G, U8 MMC5983MA, U9 XC8111, Y1 40MHz±10ppm

Commit message: Conitnued with v2, NB pinout of external sd card has changed!!! Chest needs to be updated before manufacturing!!!
Parts:
- removed C37: 100nF, Capacitor_SMD:C_0402_1005Metric
- moved C3 10.6 mm to (171.9, 80.3)
- moved C6 10.6 mm to (172.9, 80.3)
- moved R10 4.92 mm to (150.3, 89.6), turned to 0 degrees
- moved R7 3.89 mm to (150.8, 90.8), turned to 180 degrees
- moved R16 3.89 mm to (150.8, 91.8), turned to 0 degrees
- moved R2 3.89 mm to (150.8, 93.8), turned to 0 degrees
- moved R3 3.89 mm to (150.8, 92.8), turned to 0 degrees
- moved R4 3.82 mm to (150.8, 95.8), turned to 0 degrees
- moved R5 3.82 mm to (150.8, 94.8), turned to 0 degrees
- moved TP7 3.73 mm to (158.3, 93.7)
- moved TP8 3.68 mm to (160.3, 93.8)
- moved D6 3.25 mm to (159.4, 87.7)
- moved J5 3.25 mm to (156.3, 90.8)
- moved R14 3.25 mm to (156.3, 89.2)
- moved R15 3.25 mm to (162.4, 89.2)
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Connections:
- J3 pad 3: /VSPI_MOSI -> /VSPI_MISO
- J3 pad 6: /VSPI_MISO -> /VSPI_MOSI
- R10 pad 1: +12V -> +24V
- U1 pad 38: /VSPI_MOSI -> /HSPI_SCLK
- U1 pad 39: /VSPI_SCLK -> /HSPI_MOSI
- U1 pad 40: /VSPI_MISO -> /HSPI_MISO
- U1 pad 41: /HSPI_SCLK -> /VSPI_MISO
- U1 pad 42: /HSPI_MOSI -> /VSPI_SCLK
- U1 pad 43: /HSPI_MISO -> /VSPI_MOSI
Routing:
- net /SCL: track 194.5 -> 74.8 mm, vias 3 -> 2
- net /SDA: track 7.53 -> 73.4 mm, vias 0 -> 2
- net /LORA_CS: track 31.7 -> 1.26 mm
- net VBUS: track 46.9 -> 18.5 mm
- net /LORA_RESET: track 20.4 -> 1.26 mm
- net /HSPI_MISO: track 35.4 -> 52.6 mm
- net /HSPI_MOSI: track 31.2 -> 47.3 mm
- net /HSPI_SCLK: track 28.3 -> 43.3 mm
- net /VSPI_SCLK: track 47.6 -> 57.7 mm
- net /VSPI_MISO: track 51.4 -> 59.7 mm
- net Net-(J5-PadA5): track 0.00 -> 5.00 mm
- net +3V3: track 52.2 -> 48.8 mm, vias 24 -> 23
- net GND: track 67.9 -> 69.9 mm, vias 160 -> 161
- net /VSPI_MOSI: track 56.1 -> 57.8 mm
- net /SD1_CS: track 3.66 -> 2.12 mm
