File: IMU.kicad_sch (KiCad schematic)
At the start: 11 parts, among them U7 H3LIS331DLTR, U8 ICM-20608-G, U9 MMC5983MA

Commit message: working on v2
Parts:
- U7: footprint iclr:PQFN50P300X300X100-16N -> iclr:QFN300X300X100-16N
Changed lines of the file:
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@@
     (property "Reference" "U7" (id 0) (at 65.405 40.64 0))
     (property "Value" "H3LIS331DLTR" (id 1) (at 65.405 43.18 0))
-    (property "Footprint" "iclr:PQFN50P300X300X100-16N" (id 2) (at 65.405 58.42 0)
+    (property "Footprint" "iclr:QFN300X300X100-16N" (id 2) (at 65.405 58.42 0)
       (effects (font (size 1.27 1.27)) (justify left bottom) hide)
     )

Commit message: v2 time
Parts:
- C21: renamed from C11; footprint Capacitor_SMD:C_0603_1608Metric -> Capacitor_SMD:C_0402_1005Metric
- C22: renamed from C12; footprint Capacitor_SMD:C_0603_1608Metric -> Capacitor_SMD:C_0402_1005Metric
- C23: renamed from C13; footprint Capacitor_SMD:C_0603_1608Metric -> Capacitor_SMD:C_0402_1005Metric
- C24: renamed from C14; footprint Capacitor_SMD:C_0603_1608Metric -> Capacitor_SMD:C_0402_1005Metric
- C25: renamed from C15; footprint Capacitor_SMD:C_0603_1608Metric -> Capacitor_SMD:C_0402_1005Metric
- C26: renamed from C16; footprint Capacitor_SMD:C_0603_1608Metric -> Capacitor_SMD:C_0402_1005Metric
- C27: renamed from C17; footprint Capacitor_SMD:C_0603_1608Metric -> Capacitor_SMD:C_0402_1005Metric
- C28: renamed from C18; footprint Capacitor_SMD:C_0603_1608Metric -> Capacitor_SMD:C_0402_1005Metric
- renumbered U7 to U6, U8 to U7, U9 to U8
Changed lines of the file:
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@@
   (symbol (lib_id "power:GND") (at 86.36 69.85 0) (unit 1)
     (in_bom yes) (on_board yes) (fields_autoplaced)
-    (property "Reference" "#PWR067" (id 0) (at 86.36 76.2 0)
+    (property "Reference" "#PWR068" (id 0) (at 86.36 76.2 0)
       (effects (font (size 1.27 1.27)) hide)
     )
@@
   (symbol (lib_id "Device:C_Small") (at 159.385 59.69 0) (unit 1)
     (in_bom yes) (on_board yes) (fields_autoplaced)
-    (property "Reference" "C13" (id 0) (at 161.925 58.4262 0)
+    (property "Reference" "C23" (id 0) (at 161.925 58.4262 0)
       (effects (font (size 1.27 1.27)) (justify left))
     )
@@
       (effects (font (size 1.27 1.27)) (justify left))
     )
-    (property "Footprint" "Capacitor_SMD:C_0603_1608Metric" (id 2) (at 159.385 59.69 0)
+    (property "Footprint" "Capacitor_SMD:C_0402_1005Metric" (id 2) (at 159.385 59.69 0)
       (effects (font (size 1.27 1.27)) hide)
     )
@@
   (symbol (lib_id "power:GND") (at 272.415 57.15 0) (unit 1)
     (in_bom yes) (on_board yes) (fields_autoplaced)
-    (property "Reference" "#PWR077" (id 0) (at 272.415 63.5 0)
+    (property "Reference" "#PWR078" (id 0) (at 272.415 63.5 0)
       (effects (font (size 1.27 1.27)) hide)
     )
@@
   (symbol (lib_id "power:GND") (at 263.525 80.01 0) (unit 1)
     (in_bom yes) (on_board yes) (fields_autoplaced)
-    (property "Reference" "#PWR075" (id 0) (at 263.525 86.36 0)
+    (property "Reference" "#PWR076" (id 0) (at 263.525 86.36 0)
       (effects (font (size 1.27 1.27)) hide)
     )
@@
   (symbol (lib_id "Device:C_Small") (at 216.535 72.39 0) (unit 1)
     (in_bom yes) (on_board yes) (fields_autoplaced)
-    (property "Reference" "C17" (id 0) (at 219.71 71.1262 0)
+    (property "Reference" "C27" (id 0) (at 219.71 71.1262 0)
       (effects (font (size 1.27 1.27)) (justify left))
     )
@@
       (effects (font (size 1.27 1.27)) (justify left))
     )
-    (property "Footprint" "Capacitor_SMD:C_0603_1608Metric" (id 2) (at 216.535 72.39 0)
+    (property "Footprint" "Capacitor_SMD:C_0402_1005Metric" (id 2) (at 216.535 72.39 0)
       (effects (font (size 1.27 1.27)) hide)
     )
@@
   (symbol (lib_id "iclr:ICM-20608-G") (at 136.525 62.23 0) (unit 1)
     (in_bom yes) (on_board yes) (fields_autoplaced)
-    (property "Reference" "U8" (id 0) (at 136.525 41.91 0))
+    (property "Reference" "U7" (id 0) (at 136.525 41.91 0))
     (property "Value" "ICM-20608-G" (id 1) (at 136.525 44.45 0))
     (property "Footprint" "iclr:PQFN50P300X300X80-16N" (id 2) (at 136.525 62.23 0)
@@
   (symbol (lib_id "power:GND") (at 216.535 77.47 0) (unit 1)
     (in_bom yes) (on_board yes) (fields_autoplaced)
-    (property "Reference" "#PWR074" (id 0) (at 216.535 83.82 0)
+    (property "Reference" "#PWR075" (id 0) (at 216.535 83.82 0)
       (effects (font (size 1.27 1.27)) hide)
     )
@@
   (symbol (lib_id "power:+3.3V") (at 160.02 48.895 0) (unit 1)
     (in_bom yes) (on_board yes) (fields_autoplaced)
-    (property "Reference" "#PWR073" (id 0) (at 160.02 52.705 0)
+    (property "Reference" "#PWR074" (id 0) (at 160.02 52.705 0)
       (effects (font (size 1.27 1.27)) hide)
     )
@@
   (symbol (lib_id "Device:C_Small") (at 272.415 54.61 0) (unit 1)
     (in_bom yes) (on_board yes) (fields_autoplaced)
-    (property "Reference" "C18" (id 0) (at 275.59 53.3462 0)
+    (property "Reference" "C28" (id 0) (at 275.59 53.3462 0)
       (effects (font (size 1.27 1.27)) (justify left))
     )
@@
       (effects (font (size 1.27 1.27)) (justify left))
     )
-    (property "Footprint" "Capacitor_SMD:C_0603_1608Metric" (id 2) (at 272.415 54.61 0)
+    (property "Footprint" "Capacitor_SMD:C_0402_1005Metric" (id 2) (at 272.415 54.61 0)
       (effects (font (size 1.27 1.27)) hide)
     )
@@
   (symbol (lib_id "power:+3.3V") (at 87.63 46.355 0) (unit 1)
     (in_bom yes) (on_board yes) (fields_autoplaced)
-    (property "Reference" "#PWR068" (id 0) (at 87.63 50.165 0)
+    (property "Reference" "#PWR069" (id 0) (at 87.63 50.165 0)
       (effects (font (size 1.27 1.27)) hide)
     )
@@
   (symbol (lib_id "power:GND") (at 92.71 55.245 0) (unit 1)
     (in_bom yes) (on_board yes) (fields_autoplaced)
-    (property "Reference" "#PWR069" (id 0) (at 92.71 61.595 0)
+    (property "Reference" "#PWR070" (id 0) (at 92.71 61.595 0)
       (effects (font (size 1.27 1.27)) hide)
     )
@@
   (symbol (lib_id "power:GND") (at 159.385 65.405 0) (unit 1)
     (in_bom yes) (on_board yes) (fields_autoplaced)
-    (property "Reference" "#PWR072" (id 0) (at 159.385 71.755 0)
+    (property "Reference" "#PWR073" (id 0) (at 159.385 71.755 0)
       (effects (font (size 1.27 1.27)) hide)
     )
@@
   (symbol (lib_id "power:GND") (at 158.75 76.835 0) (unit 1)
     (in_bom yes) (on_board yes) (fields_autoplaced)
-    (property "Reference" "#PWR071" (id 0) (at 158.75 83.185 0)
+    (property "Reference" "#PWR072" (id 0) (at 158.75 83.185 0)
       (effects (font (size 1.27 1.27)) hide)
     )
@@
   (symbol (lib_id "Device:C_Small") (at 172.72 52.07 0) (unit 1)
     (in_bom yes) (on_board yes) (fields_autoplaced)
-    (property "Reference" "C15" (id 0) (at 175.895 50.8062 0)
+    (property "Reference" "C25" (id 0) (at 175.895 50.8062 0)
       (effects (font (size 1.27 1.27)) (justify left))
     )
@@
       (effects (font (size 1.27 1.27)) (justify left))
     )
-    (property "Footprint" "Capacitor_SMD:C_0603_1608Metric" (id 2) (at 172.72 52.07 0)
+    (property "Footprint" "Capacitor_SMD:C_0402_1005Metric" (id 2) (at 172.72 52.07 0)
       (effects (font (size 1.27 1.27)) hide)
     )
@@
   (symbol (lib_id "Device:C_Small") (at 90.805 50.8 0) (unit 1)
     (in_bom yes) (on_board yes) (fields_autoplaced)
-    (property "Reference" "C11" (id 0) (at 93.345 49.5362 0)
+    (property "Reference" "C21" (id 0) (at 93.345 49.5362 0)
       (effects (font (size 1.27 1.27)) (justify left))
     )
@@
       (effects (font (size 1.27 1.27)) (justify left))
     )
-    (property "Footprint" "Capacitor_SMD:C_0603_1608Metric" (id 2) (at 90.805 50.8 0)
+    (property "Footprint" "Capacitor_SMD:C_0402_1005Metric" (id 2) (at 90.805 50.8 0)
       (effects (font (size 1.27 1.27)) hide)
     )
@@
   (symbol (lib_id "power:+3.3V") (at 266.7 51.435 0) (unit 1)
     (in_bom yes) (on_board yes) (fields_autoplaced)
-    (property "Reference" "#PWR076" (id 0) (at 266.7 55.245 0)
+    (property "Reference" "#PWR077" (id 0) (at 266.7 55.245 0)
       (effects (font (size 1.27 1.27)) hide)
     )
@@
   (symbol (lib_id "iclr:H3LIS100DLTR") (at 65.405 58.42 0) (unit 1)
     (in_bom yes) (on_board yes) (fields_autoplaced)
-    (property "Reference" "U7" (id 0) (at 65.405 40.64 0))
+    (property "Reference" "U6" (id 0) (at 65.405 40.64 0))
     (property "Value" "H3LIS331DLTR" (id 1) (at 65.405 43.18 0))
     (property "Footprint" "iclr:QFN300X300X100-16N" (id 2) (at 65.405 58.42 0)
@@
   (symbol (lib_id "Device:C_Small") (at 95.25 50.8 0) (unit 1)
     (in_bom yes) (on_board yes) (fields_autoplaced)
-    (property "Reference" "C12" (id 0) (at 98.425 49.5362 0)
+    (property "Reference" "C22" (id 0) (at 98.425 49.5362 0)
       (effects (font (size 1.27 1.27)) (justify left))
     )
@@
       (effects (font (size 1.27 1.27)) (justify left))
     )
-    (property "Footprint" "Capacitor_SMD:C_0603_1608Metric" (id 2) (at 95.25 50.8 0)
+    (property "Footprint" "Capacitor_SMD:C_0402_1005Metric" (id 2) (at 95.25 50.8 0)
       (effects (font (size 1.27 1.27)) hide)
     )
@@
   (symbol (lib_id "iclr:MMC5983MA") (at 243.205 64.77 0) (unit 1)
     (in_bom yes) (on_board yes) (fields_autoplaced)
-    (property "Reference" "U9" (id 0) (at 243.205 43.815 0))
+    (property "Reference" "U8" (id 0) (at 243.205 43.815 0))
     (property "Value" "MMC5983MA" (id 1) (at 243.205 46.355 0))
     (property "Footprint" "iclr:PQFN50P300X300X100-16N" (id 2) (at 243.205 64.77 0)
@@
   (symbol (lib_id "Device:C_Small") (at 183.515 52.07 0) (unit 1)
     (in_bom yes) (on_board yes)
-    (property "Reference" "C16" (id 0) (at 188.595 50.8 0)
+    (property "Reference" "C26" (id 0) (at 188.595 50.8 0)
       (effects (font (size 1.27 1.27)) (justify left))
     )
@@
       (effects (font (size 1.27 1.27)) (justify left))
     )
-    (property "Footprint" "Capacitor_SMD:C_0603_1608Metric" (id 2) (at 183.515 52.07 0)
+    (property "Footprint" "Capacitor_SMD:C_0402_1005Metric" (id 2) (at 183.515 52.07 0)
       (effects (font (size 1.27 1.27)) hide)
     )
@@
   (symbol (lib_id "Device:C_Small") (at 166.37 54.61 0) (unit 1)
     (in_bom yes) (on_board yes) (fields_autoplaced)
-    (property "Reference" "C14" (id 0) (at 168.91 53.3462 0)
+    (property "Reference" "C24" (id 0) (at 168.91 53.3462 0)
       (effects (font (size 1.27 1.27)) (justify left))
     )
@@
       (effects (font (size 1.27 1.27)) (justify left))
     )
-    (property "Footprint" "Capacitor_SMD:C_0603_1608Metric" (id 2) (at 166.37 54.61 0)
+    (property "Footprint" "Capacitor_SMD:C_0402_1005Metric" (id 2) (at 166.37 54.61 0)
       (effects (font (size 1.27 1.27)) hide)
     )
@@
   (symbol (lib_id "power:GND") (at 111.76 55.245 0) (unit 1)
     (in_bom yes) (on_board yes) (fields_autoplaced)
-    (property "Reference" "#PWR070" (id 0) (at 111.76 61.595 0)
-      (effects (font (size 1.27 1.27)) hide)
-    )
+    (property "Reference" "#PWR071" (id 0) (at 111.76 61.595 0)
+      (effects (font (size 1.27 1.27)) hide)
+    )
