File: radio.kicad_sch (KiCad schematic)
At the start: 4 parts, among them J18 Conn_Coaxial, U19 RFM95W-868S2

Commit message: v2 time
Parts:
- C55: renamed from C34; footprint Capacitor_SMD:C_0603_1608Metric -> Capacitor_SMD:C_0402_1005Metric
- C56: renamed from C35; footprint Capacitor_SMD:C_0603_1608Metric -> Capacitor_SMD:C_0402_1005Metric
- renumbered J18 to J11, U19 to U21
Other:
- note added: "73251-1150"
Changed lines of the file:
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@@
     (stroke (width 0) (type default) (color 0 0 0 0))
+  )
+  (text "73251-1150" (at 170.18 96.52 0)
+    (effects (font (size 1.27 1.27)) (justify left bottom))
   )
   (hierarchical_label "~{INT}" (shape output) (at 151.13 107.315 0)
@@
   (symbol (lib_id "Device:C_Small") (at 146.05 72.39 0) (unit 1)
     (in_bom yes) (on_board yes) (fields_autoplaced)
-    (property "Reference" "C34" (id 0) (at 149.225 71.1262 0)
+    (property "Reference" "C55" (id 0) (at 149.225 71.1262 0)
       (effects (font (size 1.27 1.27)) (justify left))
     )
@@
       (effects (font (size 1.27 1.27)) (justify left))
     )
-    (property "Footprint" "Capacitor_SMD:C_0603_1608Metric" (id 2) (at 146.05 72.39 0)
+    (property "Footprint" "Capacitor_SMD:C_0402_1005Metric" (id 2) (at 146.05 72.39 0)
       (effects (font (size 1.27 1.27)) hide)
     )
@@
   (symbol (lib_id "power:GND") (at 166.37 95.885 0) (unit 1)
     (in_bom yes) (on_board yes)
-    (property "Reference" "#PWR0124" (id 0) (at 166.37 102.235 0)
+    (property "Reference" "#PWR0129" (id 0) (at 166.37 102.235 0)
       (effects (font (size 1.27 1.27)) hide)
     )
@@
   (symbol (lib_id "RF_Module:RFM95W-868S2") (at 138.43 97.155 0) (unit 1)
     (in_bom yes) (on_board yes)
-    (property "Reference" "U19" (id 0) (at 149.225 81.915 0))
+    (property "Reference" "U21" (id 0) (at 149.225 81.915 0))
     (property "Value" "RFM95W-868S2" (id 1) (at 148.59 84.455 0))
     (property "Footprint" "RF_Module:HOPERF_RFM9XW_SMD" (id 2) (at 54.61 55.245 0)
@@
   (symbol (lib_id "Connector:Conn_Coaxial") (at 166.37 89.535 0) (unit 1)
     (in_bom yes) (on_board yes)
-    (property "Reference" "J18" (id 0) (at 168.91 90.17 0)
+    (property "Reference" "J11" (id 0) (at 168.91 90.17 0)
       (effects (font (size 1.27 1.27)) (justify left))
     )
@@
   (symbol (lib_id "Device:C_Small") (at 151.13 72.39 0) (unit 1)
     (in_bom yes) (on_board yes)
-    (property "Reference" "C35" (id 0) (at 154.305 71.1262 0)
+    (property "Reference" "C56" (id 0) (at 154.305 71.1262 0)
       (effects (font (size 1.27 1.27)) (justify left))
     )
@@
       (effects (font (size 1.27 1.27)) (justify left))
     )
-    (property "Footprint" "Capacitor_SMD:C_0603_1608Metric" (id 2) (at 151.13 72.39 0)
+    (property "Footprint" "Capacitor_SMD:C_0402_1005Metric" (id 2) (at 151.13 72.39 0)
       (effects (font (size 1.27 1.27)) hide)
     )
@@
   (symbol (lib_id "power:GND") (at 148.59 74.93 0) (unit 1)
     (in_bom yes) (on_board yes) (fields_autoplaced)
-    (property "Reference" "#PWR0123" (id 0) (at 148.59 81.28 0)
+    (property "Reference" "#PWR0128" (id 0) (at 148.59 81.28 0)
       (effects (font (size 1.27 1.27)) hide)
     )
@@
   (symbol (lib_id "power:+3V3") (at 138.43 68.58 0) (unit 1)
     (in_bom yes) (on_board yes)
-    (property "Reference" "#PWR0121" (id 0) (at 138.43 72.39 0)
+    (property "Reference" "#PWR0126" (id 0) (at 138.43 72.39 0)
       (effects (font (size 1.27 1.27)) hide)
     )
@@
   (symbol (lib_id "power:GND") (at 140.97 114.935 0) (unit 1)
     (in_bom yes) (on_board yes)
-    (property "Reference" "#PWR0122" (id 0) (at 140.97 121.285 0)
+    (property "Reference" "#PWR0127" (id 0) (at 140.97 121.285 0)
       (effects (font (size 1.27 1.27)) hide)
     )
