File: power.kicad_sch (KiCad schematic)
At the start: 57 parts, among them J8 DeployLipo, J9 UCLipo, Q10 DMP3099L, Q6 SI4143DY-T1-GE3, Q7 SI4143DY-T1-GE3, Q8 DMP3099L, Q9 DMP3099L, U10 LTC4412xS6, U11 MP28167GQ-A-Z, U14 LTC4412xS6, U16 SC4215, U17 LTC4412xS6, U22 LTC4412xS6, U9 LTC4412xS6

Commit message: initial layout complete
Connections:
- net BB_IN: now also R25.1
- net GND: now also C44.2
- net UC_Lipo+: no longer R25.1
Other:
- moved on the sheet: R25, R26
Changed lines of the file:
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@@
   (junction (at 271.78 38.1) (diameter 0) (color 0 0 0 0)
   )
-  (junction (at 58.42 43.18) (diameter 0) (color 0 0 0 0)
+  (junction (at 87.63 45.72) (diameter 0) (color 0 0 0 0)
   )
   (junction (at 191.77 77.47) (diameter 0) (color 0 0 0 0)
   )
   (junction (at 24.13 62.23) (diameter 0) (color 0 0 0 0)
-  )
-  (junction (at 46.99 36.83) (diameter 0) (color 0 0 0 0)
   )
   (junction (at 111.76 160.02) (diameter 0) (color 0 0 0 0)
@@
   (no_connect (at 219.71 50.8))
   (no_connect (at 67.31 129.54))
-  (wire (pts (xy 58.42 43.18) (xy 71.12 43.18))
+  (wire (pts (xy 87.63 45.72) (xy 100.33 45.72))
     (stroke (width 0) (type default))
   )
@@
     (stroke (width 0) (type default))
   )
-  (wire (pts (xy 46.99 36.83) (xy 46.99 40.64))
+  (wire (pts (xy 46.99 30.48) (xy 46.99 40.64))
     (stroke (width 0) (type default))
   )
@@
     (stroke (width 0) (type default))
   )
+  (wire (pts (xy 87.63 36.83) (xy 87.63 39.37))
+    (stroke (width 0) (type default))
+  )
   (wire (pts (xy 38.1 160.02) (xy 46.99 160.02))
     (stroke (width 0) (type default))
@@
     (stroke (width 0) (type default))
   )
-  (wire (pts (xy 58.42 43.18) (xy 58.42 41.91))
+  (wire (pts (xy 87.63 45.72) (xy 87.63 44.45))
     (stroke (width 0) (type default))
   )
@@
     (stroke (width 0) (type default))
   )
-  (wire (pts (xy 46.99 30.48) (xy 46.99 36.83))
-    (stroke (width 0) (type default))
-  )
   (wire (pts (xy 102.87 72.39) (xy 96.52 72.39))
     (stroke (width 0) (type default))
@@
     (stroke (width 0) (type default))
   )
-  (wire (pts (xy 58.42 44.45) (xy 58.42 43.18))
+  (wire (pts (xy 87.63 46.99) (xy 87.63 45.72))
     (stroke (width 0) (type default))
   )
@@
     (stroke (width 0) (type default))
   )
-  (wire (pts (xy 46.99 36.83) (xy 58.42 36.83))
-    (stroke (width 0) (type default))
-  )
   (wire (pts (xy 123.19 99.06) (xy 120.65 99.06))
     (stroke (width 0) (type default))
@@
     (stroke (width 0) (type default))
   )
-  (wire (pts (xy 58.42 49.53) (xy 58.42 50.8))
+  (wire (pts (xy 87.63 52.07) (xy 87.63 53.34))
     (stroke (width 0) (type default))
   )
@@
   )
   (text "Allows a voltage range of up to 30v -> 80k and 10k scaled to 3.333v"
-    (at 15.24 19.05 0)
+    (at 68.58 27.94 0)
     (effects (font (size 1.27 1.27)) (justify left bottom))
   )
@@
     (effects (font (size 1.27 1.27)) (justify left bottom))
   )
+  (label "BB_IN" (at 87.63 36.83 0) (fields_autoplaced)
+    (effects (font (size 1.27 1.27)) (justify left bottom))
+  )
   (label "UC_Lipo+" (at 31.75 160.02 180) (fields_autoplaced)
     (effects (font (size 1.27 1.27)) (justify right bottom))
@@
     (effects (font (size 1.27 1.27)) (justify right))
   )
-  (hierarchical_label "UC_Lipo_Scaled" (shape output) (at 71.12 43.18 0) (fields_autoplaced)
+  (hierarchical_label "UC_Lipo_Scaled" (shape output) (at 100.33 45.72 0) (fields_autoplaced)
     (effects (font (size 1.27 1.27)) (justify left))
   )
@@
     )
   )
+  (symbol (lib_name "GND_3") (lib_id "power:GND") (at 207.01 43.18 0) (unit 1)
+    (in_bom yes) (on_board yes) (dnp no) (fields_autoplaced)
+    (property "Reference" "#PWR099" (at 207.01 49.53 0)
+      (effects (font (size 1.27 1.27)) hide)
+    )
+    (property "Value" "GND" (at 207.01 48.26 0)
+      (effects (font (size 1.27 1.27)))
+    )
+    (property "Footprint" "" (at 207.01 43.18 0)
+      (effects (font (size 1.27 1.27)) hide)
+    )
+    (property "Datasheet" "" (at 207.01 43.18 0)
+      (effects (font (size 1.27 1.27)) hide)
+    )
+    (pin "1")
+    (instances
+      (project "PickleRick"
+        (path "/e63e39d7-6ac0-4ffd-8aa3-1841a4541b55/150d7a0e-7d8c-4788-bc30-4a3682bf4d09"
+          (reference "#PWR099") (unit 1)
+        )
+      )
+    )
+  )
   (symbol (lib_name "GND_2") (lib_id "power:GND") (at 57.15 190.5 0) (unit 1)
     (in_bom yes) (on_board yes) (dnp no) (fields_autoplaced)
@@
     )
   )
-  (symbol (lib_id "Device:R_Small") (at 58.42 39.37 0) (unit 1)
-    (in_bom yes) (on_board yes) (dnp no) (fields_autoplaced)
-    (property "Reference" "R25" (at 60.96 38.0999 0)
-      (effects (font (size 1.27 1.27)) (justify left))
-    )
-    (property "Value" "80k" (at 60.96 40.6399 0)
-      (effects (font (size 1.27 1.27)) (justify left))
-    )
-    (property "Footprint" "Resistor_SMD:R_0402_1005Metric" (at 58.42 39.37 0)
-      (effects (font (size 1.27 1.27)) hide)
-    )
-    (property "Datasheet" "~" (at 58.42 39.37 0)
+  (symbol (lib_id "Device:R_Small") (at 87.63 41.91 0) (unit 1)
+    (in_bom yes) (on_board yes) (dnp no) (fields_autoplaced)
+    (property "Reference" "R25" (at 90.17 40.6399 0)
+      (effects (font (size 1.27 1.27)) (justify left))
+    )
+    (property "Value" "80k" (at 90.17 43.1799 0)
+      (effects (font (size 1.27 1.27)) (justify left))
+    )
+    (property "Footprint" "Resistor_SMD:R_0402_1005Metric" (at 87.63 41.91 0)
+      (effects (font (size 1.27 1.27)) hide)
+    )
+    (property "Datasheet" "~" (at 87.63 41.91 0)
       (effects (font (size 1.27 1.27)) hide)
     )
@@
     )
   )
-  (symbol (lib_id "power:GND") (at 58.42 50.8 0) (unit 1)
-    (in_bom yes) (on_board yes) (dnp no) (fields_autoplaced)
-    (property "Reference" "#PWR087" (at 58.42 57.15 0)
-      (effects (font (size 1.27 1.27)) hide)
-    )
-    (property "Value" "GND" (at 58.42 55.88 0)
-      (effects (font (size 1.27 1.27)))
-    )
-    (property "Footprint" "" (at 58.42 50.8 0)
-      (effects (font (size 1.27 1.27)) hide)
-    )
-    (property "Datasheet" "" (at 58.42 50.8 0)
+  (symbol (lib_id "power:GND") (at 87.63 53.34 0) (unit 1)
+    (in_bom yes) (on_board yes) (dnp no) (fields_autoplaced)
+    (property "Reference" "#PWR087" (at 87.63 59.69 0)
+      (effects (font (size 1.27 1.27)) hide)
+    )
+    (property "Value" "GND" (at 87.63 58.42 0)
+      (effects (font (size 1.27 1.27)))
+    )
+    (property "Footprint" "" (at 87.63 53.34 0)
+      (effects (font (size 1.27 1.27)) hide)
+    )
+    (property "Datasheet" "" (at 87.63 53.34 0)
       (effects (font (size 1.27 1.27)) hide)
     )
@@
     )
   )
-  (symbol (lib_id "Device:R_Small") (at 58.42 46.99 0) (unit 1)
-    (in_bom yes) (on_board yes) (dnp no) (fields_autoplaced)
-    (property "Reference" "R26" (at 60.96 45.7199 0)
-      (effects (font (size 1.27 1.27)) (justify left))
-    )
-    (property "Value" "10k" (at 60.96 48.2599 0)
-      (effects (font (size 1.27 1.27)) (justify left))
-    )
-    (property "Footprint" "Resistor_SMD:R_0402_1005Metric" (at 58.42 46.99 0)
-      (effects (font (size 1.27 1.27)) hide)
-    )
-    (property "Datasheet" "~" (at 58.42 46.99 0)
-      (effects (font (size 1.27 1.27)) hide)
-    )
+  (symbol (lib_id "Device:R_Small") (at 87.63 49.53 0) (unit 1)
+    (in_bom yes) (on_board yes) (dnp no) (fields_autoplaced)
+    (property "Reference" "R26" (at 90.17 48.2599 0)
+      (effects (font (size 1.27 1.27)) (justify left))
+    )
+    (property "Value" "10k" (at 90.17 50.7999 0)
+      (effects (font (size 1.27 1.27)) (justify left))
+    )
+    (property "Footprint" "Resistor_SMD:R_0402_1005Metric" (at 87.63 49.53 0)
+      (effects (font (size 1.27 1.27)) hide)
+    )
+    (property "Datasheet" "~" (at 87.63 49.53 0)
+      (effects (font (size 1.27 1.27)) hide)
+    )
