File: power.kicad_sch (KiCad schematic)
At the start: 57 parts, among them J8 DeployLipo, J9 UCLipo, Q10 DMP3099L, Q6 SI4143DY-T1-GE3, Q7 SI4143DY-T1-GE3, Q8 DMP3099L, Q9 DMP3099L, U10 LTC4412xS6, U11 MP28167GQ-A-Z, U14 LTC4412xS6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

Commit message: layout almost complete
Parts:
- removed J8: DeployLipo, TerminalBlock_Phoenix:TerminalBlock_Phoenix_MKDS-3-2-5.08_1x02_P5.08mm_Horizontal, symbol Connector:Conn_01x02_Male
Changed lines of the file:
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@@
   (junction (at 85.09 95.25) (diameter 0) (color 0 0 0 0)
-  )
-  (junction (at 25.4 40.64) (diameter 0) (color 0 0 0 0)
   )
   (junction (at 209.55 90.17) (diameter 0) (color 0 0 0 0)
@@
         )
       )
-    )
-  )
-  (symbol (lib_id "Connector:Conn_01x02_Male") (at 25.4 35.56 270) (unit 1)
-    (in_bom yes) (on_board yes) (dnp no) (fields_autoplaced)
-    (property "Reference" "J8" (at 26.67 34.9249 90)
-      (effects (font (size 1.27 1.27)) (justify left))
-    )
-    (property "Value" "DeployLipo" (at 26.67 37.4649 90)
-      (effects (font (size 1.27 1.27)) (justify left))
-    )
-    (property "Footprint" "TerminalBlock_Phoenix:TerminalBlock_Phoenix_MKDS-3-2-5.08_1x02_P5.08mm_Horizontal" (at 25.4 35.56 0)
-      (effects (font (size 1.27 1.27)) hide)
-    )
-    (property "Datasheet" "~" (at 25.4 35.56 0)
-      (effects (font (size 1.27 1.27)) hide)
-    )
-    (pin "1")
-    (pin "2")
-    (instances
-      (project "PickleRick"
-        (path "/e63e39d7-6ac0-4ffd-8aa3-1841a4541b55/150d7a0e-7d8c-4788-bc30-4a3682bf4d09"
-          (reference "J8") (unit 1)
-        )
-      )

Commit message: update
Parts:
- added J8: DeployLipo, TerminalBlock_Phoenix:TerminalBlock_Phoenix_MKDS-3-2-5.08_1x02_P5.08mm_Horizontal, symbol Connector:Conn_01x02_Male
Connections:
- net Deploy_Lipo+: now also J8.1 (Pin_1)
- net GND: now also J8.2 (Pin_2)
Changed lines of the file:
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@@
   (junction (at 85.09 95.25) (diameter 0) (color 0 0 0 0)
+  )
+  (junction (at 25.4 40.64) (diameter 0) (color 0 0 0 0)
   )
   (junction (at 209.55 90.17) (diameter 0) (color 0 0 0 0)
@@
         )
       )
+    )
+  )
+  (symbol (lib_id "Connector:Conn_01x02_Male") (at 25.4 35.56 270) (unit 1)
+    (in_bom yes) (on_board yes) (dnp no) (fields_autoplaced)
+    (property "Reference" "J8" (at 26.67 34.9249 90)
+      (effects (font (size 1.27 1.27)) (justify left))
+    )
+    (property "Value" "DeployLipo" (at 26.67 37.4649 90)
+      (effects (font (size 1.27 1.27)) (justify left))
+    )
+    (property "Footprint" "TerminalBlock_Phoenix:TerminalBlock_Phoenix_MKDS-3-2-5.08_1x02_P5.08mm_Horizontal" (at 25.4 35.56 0)
+      (effects (font (size 1.27 1.27)) hide)
+    )
+    (property "Datasheet" "~" (at 25.4 35.56 0)
+      (effects (font (size 1.27 1.27)) hide)
+    )
+    (pin "1")
+    (pin "2")
+    (instances
+      (project "PickleRick"
+        (path "/e63e39d7-6ac0-4ffd-8aa3-1841a4541b55/150d7a0e-7d8c-4788-bc30-4a3682bf4d09"
+          (reference "J8") (unit 1)
+        )
+      )

Commit message: update
Parts:
- C33: value 12nF -> 22nF
Changed lines of the file:
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@@
       (effects (font (size 1.27 1.27)) (justify left))
     )
-    (property "Value" "12nF" (at 128.27 103.5113 0)
+    (property "Value" "22nF" (at 128.27 103.5113 0)
       (effects (font (size 1.27 1.27)) (justify left))
     )
