File: PickleRick.kicad_pcb (KiCad board)
At the start: 4 copper layers, 100 x 37 mm, 172 parts, among them J1 RBUS, J10 Conn_Coaxial, J11 Conn_Coaxial, J12 Conn_01x03_Male, J2 Conn_01x02_Male, J3 292227-7, J4 Micro_SD_Card_Det, J5 USB_C_Receptacle_USB2.0, J6 Screw_Terminal_01x08, J7 Conn_01x05_Male, J8 DeployLipo, J9 UCLipo, Q1 PMV20ENR, Q2 NCV8415STT1G, Q3 NCV8415STT1G, Q4 NCV8415STT1G, Q5 NCV8415STT1G, Q6 SI4143DY-T1-GE3, Q7 SI4143DY-T1-GE3, U1 ESP32-S3, U10 NCP1117-3.3_SOT223, U11 XC8111, U12 XC8111, U13 XC8111, U14 LTC4412xS6, U15 MAX77827AEFD+T, U16 SC4215, U17 LTC4412xS6, U18 XC8111, U19 MAX-M10S, U2 DPS310, U20 SN65HVD230, U21 RFM95W-868S2, U3 LTV-247, U4 PCA9534RGVR, U5 PCA9685BS, U6 H3LIS331DLTR, U7 ICM-20608-G, U8 MMC5983MA, U9 XC8111, Y1 40MHz±10ppm

Commit message: did layout of buck kinda. 90% there
Parts:
- removed JP1: SolderJumper_3_Bridged12, Jumper:SolderJumper-3_P1.3mm_Bridged12_RoundedPad1.0x1.5mm
- removed TP12, TP14: TestPoint, TestPoint:TestPoint_Pad_D1.0mm
- removed U12, U13, U18: XC8111, Package_TO_SOT_SMD:SOT-23-5
- removed U15: MAX77827AEFD+T, iclr:CONV_MAX77827AEFD+T
- added C57: 22uF, Capacitor_SMD:C_0402_1005Metric, F.Cu at (188.7, 85.8)
- added Q10: DMP3099L, Package_TO_SOT_SMD:SOT-23, F.Cu at (175.1, 48.2)
- added Q8: DMP3099L, Package_TO_SOT_SMD:SOT-23, F.Cu at (171.7, 43.5)
- added Q9: DMP3099L, Package_TO_SOT_SMD:SOT-23, F.Cu at (168.2, 48.2)
- added R36: 10k, Capacitor_SMD:C_0402_1005Metric, F.Cu at (185.1, 74.7)
- added R37: 37.4k, Capacitor_SMD:C_0402_1005Metric, F.Cu at (183.9, 77.5)
- added R40: 806k, Capacitor_SMD:C_0402_1005Metric, F.Cu at (185.4, 81.0)
- added R41: 430k, Capacitor_SMD:C_0402_1005Metric, F.Cu at (184.4, 81.0)
- added R42: 143k, Capacitor_SMD:C_0402_1005Metric, F.Cu at (183.9, 79.5)
- added R43: 10k, Capacitor_SMD:C_0402_1005Metric, F.Cu at (183.4, 75.3)
- added R44: 10k, Capacitor_SMD:C_0402_1005Metric, F.Cu at (183.4, 76.2)
- added TP16: TestPoint, TestPoint:TestPoint_Pad_D1.0mm, F.Cu at (181.4, 74.8)
- added TP17: TestPoint, TestPoint:TestPoint_Pad_D1.0mm, F.Cu at (181.4, 76.8)
- added U22: LTC4412xS6, Package_TO_SOT_SMD:TSOT-23-6, F.Cu at (178.7, 48.3)
- C30: value 0.1uF -> 22nF
- C32: value 10uF -> 1uF
- C33: value 10uF -> 12nF
- C36: value 0.1uF -> 22uF; footprint Capacitor_SMD:C_0402_1005Metric -> Capacitor_SMD:C_0805_2012Metric
- C38: value 0.1uF -> 100uF; footprint Capacitor_SMD:C_0402_1005Metric -> Capacitor_SMD:CP_Elec_6.3x9.9
- C39: value 10uF -> 100nF; footprint Capacitor_SMD:C_0603_1608Metric -> Capacitor_SMD:C_0402_1005Metric
- C40: value 1uF -> 100nF
- C42: footprint Capacitor_SMD:C_0603_1608Metric -> Capacitor_SMD:C_0402_1005Metric
- C43: value 10uF -> 22uF
- C47, C48: value 0.1uF -> 22uF
- L3: value 1uH -> MPL-AL6050-4R7; footprint Inductor_SMD:L_0805_2012Metric -> iclr:MPLAL60504R7
- R25: value 51k -> 80k
- R27: value 14k -> 499k; footprint Resistor_SMD:R_0402_1005Metric -> Capacitor_SMD:C_0402_1005Metric
- TP10, TP11, TP13: footprint TestPoint:TestPoint_Pad_D1.0mm -> TestPoint:TestPoint_Pad_D2.0mm
- U10: value NCP1117-3.3_SOT223 -> LTC4412xS6; footprint Package_TO_SOT_SMD:SOT-223-3_TabPin2 -> Package_TO_SOT_SMD:TSOT-23-6
- U11: value XC8111 -> QFN-16_MP28167_MNP; footprint Package_TO_SOT_SMD:SOT-23-5 -> iclr:MP28167GQ-A-Z
- U9: value XC8111 -> LTC4412xS6; footprint Package_TO_SOT_SMD:SOT-23-5 -> Package_TO_SOT_SMD:TSOT-23-6
- moved TP11 60.9 mm to (225.0, 53.0)
- moved U9 49.1 mm to (168.2, 43.3), turned to -90 degrees
- moved C35 48.8 mm to (168.7, 40.8), turned to 180 degrees
- moved C31 48.6 mm to (179.3, 43.7), turned to 180 degrees
- moved TP13 41.1 mm to (231.8, 52.9)
- moved U10 24.5 mm to (171.7, 48.4), turned to 90 degrees
- moved TP10 23.3 mm to (196.7, 69.1), turned to -90 degrees
- moved C30 19.1 mm to (186.4, 74.2), turned to 90 degrees
- moved U11 18.9 mm to (188.2, 78.3), turned to -90 degrees
- moved C29 18.4 mm to (171.2, 50.9), turned to 0 degrees
- moved C36 16.4 mm to (188.6, 73.8), turned to 180 degrees
- moved C34 16.4 mm to (188.7, 75.3), turned to 180 degrees
- moved C44 13.6 mm to (189.3, 87.4), turned to -90 degrees
- moved C43 10.8 mm to (188.7, 82.8), turned to 180 degrees
- moved C32 10.6 mm to (187.1, 81.3), turned to -90 degrees
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Connections:
- C29 pad 1: Net-(C29-Pad1) -> /power/RBUS_3.3V_IN
- C30 pad 1: /power/RBUS_3.3V_IN -> Net-(U11-EN)
- C32 pad 1: GND -> /power/BB_VCC
- C32 pad 2: Net-(C32-Pad2) -> GND
- C33 pad 1: GND -> Net-(U11-OC)
- C33 pad 2: Net-(C33-Pad2) -> GND
- C34 pad 1: /power/BBIN -> /power/BB_IN
- C35 pad 1: /power/BBIN -> /power/UC_Lipo+
- C36 pad 1: /power/BBIN -> /power/BB_IN
- C38 pad 1: GND -> /power/BB_IN
- C38 pad 2: Net-(C33-Pad2) -> GND
- C39 pad 1: /power/BBIN -> Net-(U11-BST1)
- C39 pad 2: GND -> Net-(U11-SW1)
- C40 pad 1: /power/BIAS -> Net-(U11-BST2)
- C40 pad 2: GND -> Net-(U11-SW2)
- C41 pad 1: +3V3 -> /power/BB_OUT
- C42 pad 1: /power/BBOUT -> /power/BB_OUT
- C43 pad 1: /power/BBOUT -> /power/BB_OUT
- C44 pad 1: /power/BBOUT -> /power/BB_OUT
- C44 pad 2: GND -> unconnected-(C44-Pad2)
- C45 pad 2: Net-(C45-Pad2) -> +3V3
- C46 pad 2: Net-(C45-Pad2) -> +3V3
- C47 pad 1: GND -> /power/BB_OUT
- C47 pad 2: Net-(C45-Pad2) -> GND
- C48 pad 1: +3V3 -> /power/BB_OUT
- L3 pad 1: /power/LX1 -> Net-(U11-SW1)
- L3 pad 2: /power/LX2 -> Net-(U11-SW2)
- R27 pad 1: /power/SEL -> /power/BB_IN
- R27 pad 2: GND -> Net-(U11-EN)
- R28 pad 1: Net-(C45-Pad2) -> +3V3
- TP10 pad 1: /power/BBIN -> /power/BB_IN
- TP11 pad 1: /power/RBUS_3.3V_IN -> +3V3
- TP13 pad 1: /power/BBOUT -> /power/BB_OUT
- U10 pad 1: GND -> /power/RBUS_3.3V_IN
- U10 pad 2: Net-(C33-Pad2) -> GND
- U10 pad 3: Net-(C32-Pad2) -> GND
- U11 pad 1: /power/RBUS_3.3V_IN -> /power/BB_IN
- U11 pad 3: /power/RBUS_3.3V_IN -> Net-(U11-EN)
- U11 pad 4: unconnected-(U11-Pad4) -> /power/BB_ALT
- U11 pad 5: /power/BBIN -> /power/BB_SCL
- U16 pad 2: /power/BBOUT -> /power/BB_OUT
- U16 pad 3: /power/BBOUT -> /power/BB_OUT
- U16 pad 6: Net-(C45-Pad2) -> +3V3
- U9 pad 1: VBUS -> /power/UC_Lipo+
- U9 pad 3: VBUS -> GND
- U9 pad 5: /power/BBIN -> Net-(Q8-G)
Routing:
- net /power/BBIN: track 38.6 -> 0.00 mm
- net GND: track 90.1 -> 73.6 mm, vias 220 -> 208
- net Net-(C33-Pad2): track 13.6 -> 0.00 mm
- net /power/BBOUT: track 12.3 -> 0.00 mm
- net /power/BB_VCC: track 0.00 -> 12.2 mm, vias 0 -> 2
- net Net-(C32-Pad2): track 11.8 -> 0.00 mm
- net VBUS: track 64.4 -> 54.3 mm, vias 4 -> 3
- net /BattVolt: track 21.8 -> 12.0 mm
- net /power/RBUS_3.3V_IN: track 18.0 -> 10.1 mm
- net Net-(C29-Pad1): track 6.99 -> 0.00 mm
- net /power/BB_SDA: track 0.00 -> 6.71 mm
- net /power/BB_SCL: track 0.00 -> 6.67 mm
- net Net-(C45-Pad2): track 6.29 -> 0.00 mm
- net +3V3: track 62.4 -> 56.8 mm, vias 39 -> 32
- net Net-(J2-Pin_1): track 6.55 -> 2.17 mm
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- added copper zone on F.Cu, net +3V3
- added copper zone on F.Cu, net /power/BB_IN
- added copper zone on F.Cu, net /power/BB_OUT
- added copper zone on F.Cu, net Net-(U11-SW1)
- added copper zone on F.Cu, net Net-(U11-SW2)
- removed copper zone on F.Cu, net (none)
- removed copper zone on F.Cu, net /power/BBOUT
- removed copper zone on B.Cu, net /power/LX1
- removed copper zone on F.Cu, net /power/LX1
- removed copper zone on B.Cu, net /power/LX2
- removed copper zone on F.Cu, net /power/LX2
- removed copper zone on F.Cu, net Net-(C45-Pad2)
Other:
- board size 100 x 37 mm -> 146.2 x 37 mm

Commit message: layout almost complete
Parts:
- added TP12: TestPoint, TestPoint:TestPoint_Pad_D1.0mm, F.Cu at (170.4, 93.0)
- added TP14: TestPoint, TestPoint:TestPoint_Pad_D1.0mm, F.Cu at (172.4, 93.0)
- added TP18: TestPoint, TestPoint:TestPoint_Pad_D1.0mm, F.Cu at (174.4, 93.0)
- added TP19: TestPoint, TestPoint:TestPoint_Pad_D1.0mm, F.Cu at (176.0, 94.2)
- added TP20: TestPoint, TestPoint:TestPoint_Pad_D1.0mm, F.Cu at (178.0, 94.2)
- added TP21: TestPoint, TestPoint:TestPoint_Pad_D1.0mm, F.Cu at (180.0, 94.2)
- added TP22: TestPoint, TestPoint:TestPoint_Pad_D1.0mm, F.Cu at (154.2, 94.5)
- added TP23: TestPoint, TestPoint:TestPoint_Pad_D1.0mm, F.Cu at (154.2, 92.5)
- added TP25: TestPoint, TestPoint:TestPoint_Pad_D1.0mm, F.Cu at (161.1, 81.6)
- added TP26: TestPoint, TestPoint:TestPoint_Pad_D1.0mm, F.Cu at (153.1, 85.2)
- added TP27: TestPoint, TestPoint:TestPoint_Pad_D1.0mm, F.Cu at (151.0, 85.2)
- added TP28: TestPoint, TestPoint:TestPoint_Pad_D1.0mm, F.Cu at (153.2, 87.7)
- Q1, R11: moved to B.Cu
- U11: value QFN-16_MP28167_MNP -> MP28167GQ-A-Z
- moved TP13 58.1 mm to (186.5, 89.2)
- moved TP11 50.1 mm to (192.7, 91.3)
- moved C31 31.0 mm to (176.5, 74.6), turned to 90 degrees
- moved Q10 25.6 mm to (178.8, 73.6)
- moved U9 24.2 mm to (177.4, 65.8)
- moved C35 24.1 mm to (174.4, 64.2), turned to 0 degrees
- moved U22 23.6 mm to (182.2, 71.7)
- moved Q8 23.2 mm to (174.0, 66.6)
- moved Q9 22.6 mm to (168.8, 70.8), turned to 180 degrees
- moved U10 19.2 mm to (168.7, 67.3), turned to 0 degrees
- moved C29 16.4 mm to (166.2, 66.5), turned to -90 degrees
- moved R25 8.65 mm to (170.6, 73.5), turned to -90 degrees
- moved Q1 8.48 mm to (187.4, 65.4)
- moved R11 8.08 mm to (189.8, 66.1)
- moved TP8 7.74 mm to (168.3, 88.8)
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Connections:
- C44 pad 2: unconnected-(C44-Pad2) -> GND
- R25 pad 1: /power/UC_Lipo+ -> /power/BB_IN
Routing:
- net VBUS: track 54.3 -> 88.7 mm
- net GND: track 73.6 -> 88.4 mm, vias 208 -> 234
- net /power/BB_IN: track 1.26 -> 13.4 mm
- net /power/UC_Lipo+: track 7.88 -> 18.3 mm
- net +3V3: track 56.8 -> 62.7 mm, vias 32 -> 40
- net Net-(Q8-G): track 0.00 -> 5.77 mm
- net /power/BB_OUT: track 1.27 -> 7.01 mm
- net /power/BB_VCC: track 12.2 -> 17.9 mm
- net Net-(Q9-G): track 0.00 -> 5.69 mm
- net /power/RBUS_3.3V_IN: track 10.1 -> 14.7 mm
- net /VSPI_MISO: track 65.8 -> 70.4 mm
- net /MAG_CS: track 28.8 -> 33.1 mm
- net /VSPI_SCLK: track 63.9 -> 68.0 mm
- net /SDA: track 134.7 -> 138.7 mm, vias 2 -> 4
- net Net-(U11-EN): track 3.93 -> 7.87 mm
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Other:
- board size 146.2 x 37 mm -> 100 x 37 mm

Commit message: update
Parts:
- added G***: LOGO, iclr:iclr_logo_estd2018_10mm, F.Cu at (129.4, 74.5)
- added G***: LOGO, iclr:pickle_ric, B.Cu at (159.2, 79.8)
- added REF**: Write_Pad, iclr:Write_Pad, F.Cu at (182.7, 79.1)
- moved R11 1.30 mm to (190.1, 64.9), turned to -90 degrees
- moved Q1 0.31 mm to (187.7, 65.4)
Routing:
- net +3V3: track 62.7 -> 64.9 mm
Other:
- board text removed: "TERM"

Commit message: almost done
Parts:
- moved TP9 14.7 mm to (153.3, 89.8)
- moved TP11 6.62 mm to (186.2, 89.9)
- moved TP25 4.97 mm to (160.0, 76.8)
- moved C56 4.97 mm to (108.1, 90.3), turned to -90 degrees
- moved C55 4.37 mm to (108.2, 88.5), turned to 90 degrees
- moved R12 3.34 mm to (149.0, 96.0)
- moved R13 3.34 mm to (149.0, 95.0)
- moved TP28 3.24 mm to (156.3, 87.2)
- moved TP13 3.13 mm to (186.3, 86.1)
- moved JP2 2.74 mm to (169.2, 66.8)
- moved J9 2.29 mm to (169.8, 63.3), turned to 180 degrees
- moved J2 2.27 mm to (190.6, 63.4), turned to 180 degrees
- moved Q1 1.85 mm to (186.1, 66.3)
- moved R11 1.85 mm to (188.6, 65.8)
- moved TP23 0.85 mm to (153.4, 92.5)
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Routing:
- net /IMU2_CS: track 15.2 -> 20.4 mm
- net +3V3: track 64.9 -> 69.1 mm, vias 40 -> 36
- net /SD1_DET: track 97.0 -> 93.5 mm
- net /SD2_DET: track 97.3 -> 94.0 mm
- net /power/UC_Lipo+: track 18.3 -> 15.0 mm
- net /power/BB_OUT: track 7.01 -> 4.47 mm
- net VBUS: track 88.7 -> 86.3 mm
- net /power/Deploy_Lipo+: track 29.4 -> 31.8 mm
- net /Buzzer: track 25.4 -> 23.7 mm
- net /LORA_INT: track 87.7 -> 86.3 mm
- net /LORA_CS: track 55.5 -> 56.7 mm
- net /nukes/Nuke1: track 35.9 -> 34.7 mm
- net /CHIP_PU: track 29.0 -> 27.8 mm
- net Net-(J2-Pin_1): track 4.65 -> 5.67 mm
- net /BARO_CS: track 32.9 -> 32.0 mm
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Other:
- board text added: "3v3"
- board text added: "4-1"
- board text added: "BB"
- board text added: "BIN"
- board text added: "BOOT"
- board text added: "BOUT"
- board text added: "EN"
- board text added: "JTAG"
- board text added: "SPI2"
- board text added: "SPI3"
- board text added: "TERM"
- board text added: "scl"
- board text added: "sda"
- board text added: "|MO|MI|SC|"
- board text added: "|MO|SC|MI|"
- board text removed: "CRX"
- board text removed: "CTX"
- board text removed: "DTR"
- board text removed: "EN BOOT"
- board text removed: "H_MISO"
- board text removed: "H_MOSI"
- board text removed: "H_SCLK"
- board text removed: "RTS"
- board text removed: "SCL"
- board text removed: "SD2"
- board text removed: "SDA"
- board text removed: "V_MISO"
- board text removed: "V_MOSI"
- board text removed: "V_SCLK"
