File: PickleRick.kicad_pcb (KiCad board)
At the start: 4 copper layers, 100 x 37 mm, 194 parts, among them J1 RBUS, J10 Conn_Coaxial, J11 Conn_Coaxial, J12 Conn_01x03_Male, J2 Conn_01x02_Male, J3 292227-7, J4 Micro_SD_Card_Det, J5 USB_C_Receptacle_USB2.0, J6 Screw_Terminal_01x08, J7 Conn_01x05_Male, J8 DeployLipo, J9 UCLipo, Q1 PMV20ENR, Q10 DMP3099L, Q2 NCV8415STT1G, Q3 NCV8415STT1G, Q4 NCV8415STT1G, Q5 NCV8415STT1G, Q6 SI4143DY-T1-GE3, Q7 SI4143DY-T1-GE3, Q8 DMP3099L, Q9 DMP3099L, U1 ESP32-S3, U10 LTC4412xS6, U11 MP28167GQ-A-Z, U14 LTC4412xS6, U16 SC4215, U17 LTC4412xS6, U19 MAX-M10S, U2 DPS310, U20 SN65HVD230, U21 RFM95W-868S2, U22 LTC4412xS6, U3 LTV-247, U4 PCA9534RGVR, U5 PCA9685BS, U6 H3LIS331DLTR, U7 ICM-20608-G, U8 MMC5983MA, U9 LTC4412xS6, Y1 40MHz±10ppm

Commit message: imagine fixing your DRC errors
Parts:
- C12: value 4.2pF -> DNP
- C13, C14: value C -> 11pF
- R8: value 47.5 -> DNP
- Y1: value 40MHz±10ppm -> R940000171
Routing:
- net GND: vias 247 -> 246
Other:
- board text added: "µPWR"
- board text removed: "uPWR"

Commit message: fixed some stuff
Routing:
- net Net-(C8-Pad1): track 3.10 -> 4.21 mm
- net GND: track 102.1 -> 102.7 mm, vias 246 -> 247
Changed lines of the file:
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@@
   (segment (start 158.2 78.941772) (end 157.904511 79.237261) (width 0.2) (layer "F.Cu") (net 1))
   (segment (start 147.962252 87.887749) (end 148.337749 87.512252) (width 0.15) (layer "F.Cu") (net 1))
+  (segment (start 117.28 68.47) (end 114.52 65.71) (width 0.4) (layer "F.Cu") (net 1))
   (segment (start 165.5 82.9) (end 165.736197 83.136197) (width 0.15) (layer "F.Cu") (net 1))
   (segment (start 177.824511 82.375489) (end 177.541318 82.375489) (width 0.4) (layer "F.Cu") (net 1))
-  (segment (start 177.9 87.2) (end 178.43 87.2) (width 0.15) (layer "F.Cu") (net 1))
+  (segment (start 177.9 87.2) (end 178.43 87.2) (width 0.2) (layer "F.Cu") (net 1))
   (segment (start 150.98 82.577276) (end 150.98 83) (width 0.15) (layer "F.Cu") (net 1))
   (segment (start 145.5 80.59) (end 145.5 80.23) (width 0.1) (layer "F.Cu") (net 1))
-  (segment (start 114.52 64.52646) (end 114.52 65.71) (width 0.15) (layer "F.Cu") (net 1))
+  (segment (start 114.52 64.52646) (end 114.52 65.71) (width 0.4) (layer "F.Cu") (net 1))
   (segment (start 186.3 91.2) (end 186.3 89.95) (width 0.2) (layer "F.Cu") (net 1))
   (segment (start 158.2 78.9) (end 158.35 78.75) (width 0.2) (layer "F.Cu") (net 1))
   (segment (start 150.98 83) (end 150.98 81.585) (width 0.15) (layer "F.Cu") (net 1))
-  (segment (start 115.46 66.62) (end 115.43 66.62) (width 0.2) (layer "F.Cu") (net 1))
   (segment (start 195.135 88.16) (end 196.743409 88.16) (width 0.9) (layer "F.Cu") (net 1))
-  (segment (start 178.43 87.2) (end 178.6 87.37) (width 0.15) (layer "F.Cu") (net 1))
+  (segment (start 178.43 87.2) (end 178.6 87.37) (width 0.2) (layer "F.Cu") (net 1))
   (segment (start 174.35 78.3) (end 174.35 78.72) (width 0.2) (layer "F.Cu") (net 1))
-  (segment (start 121.36 70.67) (end 121.36 68.47) (width 0.2) (layer "F.Cu") (net 1))
+  (segment (start 121.36 70.67) (end 121.36 68.47) (width 0.4) (layer "F.Cu") (net 1))
   (segment (start 178.12 81.8) (end 178.12 81.662784) (width 0.4) (layer "F.Cu") (net 1))
   (segment (start 185.2 89.9) (end 185 89.7) (width 0.2) (layer "F.Cu") (net 1))
-  (segment (start 117.31 68.47) (end 115.46 66.62) (width 0.2) (layer "F.Cu") (net 1))
   (segment (start 111.25 64.95) (end 111.25 65.71) (width 0.15) (layer "F.Cu") (net 1))
   (segment (start 150.511478 81.243427) (end 150.174905 81.58) (width 0.15) (layer "F.Cu") (net 1))
@@
   (segment (start 108.61 89.35) (end 108.14 89.82) (width 0.4) (layer "F.Cu") (net 1))
   (segment (start 108.65 89.35) (end 108.61 89.35) (width 0.4) (layer "F.Cu") (net 1))
-  (segment (start 169.225 85.2) (end 169.955 85.2) (width 0.15) (layer "F.Cu") (net 1))
+  (segment (start 169.225 85.2) (end 169.955 85.2) (width 0.2) (layer "F.Cu") (net 1))
   (segment (start 169.99 90.57) (end 170.32 90.9) (width 0.2) (layer "F.Cu") (net 1))
   (segment (start 158.35 78.75) (end 158.35 78.3) (width 0.2) (layer "F.Cu") (net 1))
@@
   (segment (start 158.47 79.17) (end 158.47 79.53) (width 0.2) (layer "F.Cu") (net 1))
   (segment (start 148.142749 88.068246) (end 148.142749 88.437749) (width 0.15) (layer "F.Cu") (net 1))
-  (segment (start 174.22 78.85) (end 174.22 79.795) (width 0.2) (layer "F.Cu") (net 1))
+  (segment (start 174.22 78.85) (end 174.22 79.795) (width 0.4) (layer "F.Cu") (net 1))
   (segment (start 178.12 81.662784) (end 178.480035 81.302749) (width 0.4) (layer "F.Cu") (net 1))
   (segment (start 186.25 89.9) (end 185.2 89.9) (width 0.2) (layer "F.Cu") (net 1))
@@
   (segment (start 150.975 81.58) (end 151.86 81.58) (width 0.15) (layer "F.Cu") (net 1))
   (segment (start 163.5 86.3) (end 163.13 85.93) (width 0.15) (layer "F.Cu") (net 1))
-  (segment (start 168.55 85.875) (end 168.55 85.475) (width 0.15) (layer "F.Cu") (net 1))
+  (segment (start 168.55 85.875) (end 168.55 85.475) (width 0.2) (layer "F.Cu") (net 1))
   (segment (start 108.675 89.375) (end 108.65 89.35) (width 0.4) (layer "F.Cu") (net 1))
-  (segment (start 168.55 85.475) (end 168.425 85.35) (width 0.15) (layer "F.Cu") (net 1))
-  (segment (start 176.845 87.2) (end 177.9 87.2) (width 0.15) (layer "F.Cu") (net 1))
+  (segment (start 168.55 85.475) (end 168.425 85.35) (width 0.2) (layer "F.Cu") (net 1))
+  (segment (start 176.845 87.2) (end 177.9 87.2) (width 0.2) (layer "F.Cu") (net 1))
   (segment (start 187.3 89.9) (end 186.25 89.9) (width 0.2) (layer "F.Cu") (net 1))
   (segment (start 150.05 81.58) (end 150.975 81.58) (width 0.15) (layer "F.Cu") (net 1))
@@
   (segment (start 151.94 82) (end 152.2 82.26) (width 0.15) (layer "F.Cu") (net 1))
   (segment (start 145.5 80.23) (end 146.455 80.23) (width 0.15) (layer "F.Cu") (net 1))
-  (segment (start 115.43 66.62) (end 114.52 65.71) (width 0.2) (layer "F.Cu") (net 1))
-  (segment (start 121.36 68.47) (end 117.31 68.47) (width 0.2) (layer "F.Cu") (net 1))
   (segment (start 165.736197 83.136197) (end 165.736197 84.15048) (width 0.15) (layer "F.Cu") (net 1))
   (segment (start 147.5 82.275) (end 147.5 81.6) (width 0.15) (layer "F.Cu") (net 1))
-  (segment (start 168.55 85.875) (end 169.225 85.2) (width 0.15) (layer "F.Cu") (net 1))
+  (segment (start 168.55 85.875) (end 169.225 85.2) (width 0.2) (layer "F.Cu") (net 1))
   (segment (start 176.845 83.071807) (end 176.845 83.49048) (width 0.4) (layer "F.Cu") (net 1))
   (segment (start 178.12 81.8) (end 178.12 82.08) (width 0.4) (layer "F.Cu") (net 1))
@@
   (segment (start 156.398341 79.898341) (end 156.5 80) (width 0.15) (layer "F.Cu") (net 1))
   (segment (start 111.25 65.71) (end 111.24 65.72) (width 0.15) (layer "F.Cu") (net 1))
+  (segment (start 121.36 68.47) (end 117.28 68.47) (width 0.4) (layer "F.Cu") (net 1))
   (segment (start 190.175 91.915) (end 190.175 91.6) (width 0.1) (layer "F.Cu") (net 1))
   (segment (start 157.904511 79.237261) (end 157.904511 79.464511) (width 0.2) (layer "F.Cu") (net 1))
@@
   (segment (start 181.55 82.95) (end 181.55 83.7) (width 0.4) (layer "F.Cu") (net 2))
   (segment (start 146.7375 76.6) (end 146.7375 75.65) (width 0.15) (layer "F.Cu") (net 2))
+  (segment (start 157.39 78.3) (end 157.39 78.88) (width 0.15) (layer "F.Cu") (net 2))
   (segment (start 147.312749 87.887749) (end 146.887749 87.462749) (width 0.15) (layer "F.Cu") (net 2))
   (segment (start 179.1255 88.15) (end 178.9455 88.33) (width 0.15) (layer "F.Cu") (net 2))
@@
   (via (at 154.035679 90.743726) (size 0.45) (drill 0.3) (layers "F.Cu" "B.Cu") (net 2))
   (via (at 162.513752 86.323067) (size 0.45) (drill 0.3) (layers "F.Cu" "B.Cu") (net 2))
+  (via (at 157.39 78.88) (size 0.45) (drill 0.3) (layers "F.Cu" "B.Cu") (net 2))
   (via (at 107.166867 83.51505) (size 0.7) (drill 0.45) (layers "F.Cu" "B.Cu") (free) (net 2))
   (via (at 142.6 78.4) (size 0.8) (drill 0.5) (layers "F.Cu" "B.Cu") (free) (net 2))
@@
   (segment (start 178.369776 85.65048) (end 186.119296 93.4) (width 0.15) (layer "B.Cu") (net 7))
   (segment (start 186.119296 93.4) (end 190.275 93.4) (width 0.15) (layer "B.Cu") (net 7))
-  (segment (start 175.28 80.78) (end 175.6 81.1) (width 0.15) (layer "F.Cu") (net 8))
-  (segment (start 175.6 82.355) (end 175.2 82.355) (width 0.15) (layer "F.Cu") (net 8))
-  (segment (start 175.2 80.78) (end 174.205 80.78) (width 0.15) (layer "F.Cu") (net 8))
-  (segment (start 175.6 81.1) (end 175.6 82.355) (width 0.15) (layer "F.Cu") (net 8))
+  (segment (start 175.28 80.78) (end 175.26 80.76) (width 0.4) (layer "F.Cu") (net 8))
+  (segment (start 175.2 80.78) (end 175.54 81.12) (width 0.4) (layer "F.Cu") (net 8))
+  (segment (start 175.26 80.76) (end 175.26 82.295) (width 0.4) (layer "F.Cu") (net 8))
+  (segment (start 175.2 80.78) (end 174.205 80.78) (width 0.4) (layer "F.Cu") (net 8))
+  (segment (start 175.54 81.12) (end 175.54 82.295) (width 0.4) (layer "F.Cu") (net 8))
   (segment (start 176.8 78.22) (end 177.77 78.22) (width 0.15) (layer "F.Cu") (net 9))
   (segment (start 181.55 85.1) (end 181.55 84.55) (width 0.1) (layer "F.Cu") (net 10))

Commit message: update
Routing:
- net GND: track 102.7 -> 97.2 mm, vias 247 -> 249
- net Net-(J5-CC2): track 6.45 -> 7.09 mm
