File: _autosave-can.kicad_sch (KiCad schematic)
At the start: 11 parts, among them U20 SN65HVD230

Commit message: update
Parts:
- R32, R33: footprint Resistor_SMD:R_0402_1005Metric -> Resistor_SMD:R_0603_1608Metric
Changed lines of the file:
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@@
       (effects (font (size 1.27 1.27)) (justify left))
     )
-    (property "Footprint" "Resistor_SMD:R_0402_1005Metric" (at 165.862 93.98 90)
+    (property "Footprint" "Resistor_SMD:R_0603_1608Metric" (at 165.862 93.98 90)
       (effects (font (size 1.27 1.27)) hide)
     )
@@
       (effects (font (size 1.27 1.27)) (justify left))
     )
-    (property "Footprint" "Resistor_SMD:R_0402_1005Metric" (at 165.862 83.82 90)
+    (property "Footprint" "Resistor_SMD:R_0603_1608Metric" (at 165.862 83.82 90)
       (effects (font (size 1.27 1.27)) hide)
     )
