File: Hardware/PickleRick.kicad_sch (KiCad schematic)
At the start: 68 parts, among them J1 RBUS, J12 Conn_01x03_Male, J2 Conn_01x02_Male, J3 292227-7, J4 Micro_SD_Card_Det, Q1 PMV20ENR, U1 ESP32-S3, U2 DPS310, Y1 R940000171

Commit message: black edition ordering stuff
Parts:
- 12VLED1: value 12V_LED -> RED_LED
- D1: value RX_LED -> ORANGE_LED
- D2: value TX_LED -> GREEN_LED
- D3: value SD1_LED -> EMERALD_LED
- D4: value SD2_LED -> GREEN_LED
- D5: value PWR_LED -> BLUE_LED
- R10: value 5k -> 5.1k; footprint Resistor_SMD:R_0603_1608Metric -> Resistor_SMD:R_0402_1005Metric
Changed lines of the file:
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@@
   )
   (symbol (lib_id "Device:C_Small") (at 274.32 113.03 0) (unit 1)
-    (in_bom yes) (on_board yes) (dnp no) (fields_autoplaced)
-    (property "Reference" "C16" (at 276.86 111.7662 0)
-      (effects (font (size 1.27 1.27)) (justify left))
-    )
-    (property "Value" "100nF" (at 276.86 114.3062 0)
+    (in_bom yes) (on_board yes) (dnp no)
+    (property "Reference" "C16" (at 279.4 111.76 0)
+      (effects (font (size 1.27 1.27)) (justify left))
+    )
+    (property "Value" "100nF" (at 279.4 114.3 0)
       (effects (font (size 1.27 1.27)) (justify left))
     )
@@
       (effects (font (size 1.27 1.27)))
     )
-    (property "Value" "TX_LED" (at 27.94 32.1056 0)
+    (property "Value" "GREEN_LED" (at 27.94 32.1056 0)
       (effects (font (size 1.27 1.27)))
     )
@@
   )
   (symbol (lib_id "Device:L") (at 39.37 135.89 90) (unit 1)
-    (in_bom yes) (on_board yes) (dnp no) (fields_autoplaced)
+    (in_bom yes) (on_board yes) (dnp no)
     (property "Reference" "L1" (at 39.37 129.54 90)
       (effects (font (size 1.27 1.27)))
@@
       (effects (font (size 1.27 1.27)))
     )
-    (property "Value" "PWR_LED" (at 57.15 17.4244 0)
+    (property "Value" "BLUE_LED" (at 57.15 17.4244 0)
       (effects (font (size 1.27 1.27)))
     )
@@
       (effects (font (size 1.27 1.27)))
     )
-    (property "Value" "SD2_LED" (at 27.94 49.2506 0)
+    (property "Value" "GREEN_LED" (at 27.94 49.2506 0)
       (effects (font (size 1.27 1.27)))
     )
@@
       (effects (font (size 1.27 1.27)))
     )
-    (property "Value" "RX_LED" (at 27.94 23.2156 0)
+    (property "Value" "ORANGE_LED" (at 27.94 23.2156 0)
       (effects (font (size 1.27 1.27)))
     )
@@
       (effects (font (size 1.27 1.27)))
     )
-    (property "Value" "SD1_LED" (at 27.94 40.9956 0)
+    (property "Value" "EMERALD_LED" (at 27.94 40.9956 0)
       (effects (font (size 1.27 1.27)))
     )
@@
       (effects (font (size 1.27 1.27)))
     )
-    (property "Value" "12V_LED" (at 66.04 23.2156 0)
+    (property "Value" "RED_LED" (at 66.04 23.2156 0)
       (effects (font (size 1.27 1.27)))
     )
@@
       (effects (font (size 1.27 1.27)))
     )
-    (property "Value" "5k" (at 71.12 17.653 90)
-      (effects (font (size 1.27 1.27)))
-    )
-    (property "Footprint" "Resistor_SMD:R_0603_1608Metric" (at 71.12 20.32 0)
-      (effects (font (size 1.27 1.27)) hide)
-    )
+    (property "Value" "5.1k" (at 71.12 17.653 90)
+      (effects (font (size 1.27 1.27)))
+    )
+    (property "Footprint" "Resistor_SMD:R_0402_1005Metric" (at 71.12 20.32 0)
+      (effects (font (size 1.27 1.27)) hide)
+    )

Commit message: 3D update
Parts:
- 12VLED1: footprint Resistor_SMD:R_0402_1005Metric -> LED_SMD:LED_0402_1005Metric
Changed lines of the file:
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@@
       (effects (font (size 1.27 1.27)))
     )
-    (property "Footprint" "Resistor_SMD:R_0402_1005Metric" (at 66.04 20.32 90)
+    (property "Footprint" "LED_SMD:LED_0402_1005Metric" (at 66.04 20.32 90)
       (effects (font (size 1.27 1.27)) hide)
     )

Commit message: v3 hardware start
Parts:
- added BZ1: CMT-0525-75-SMT-TR, symbol Device:Buzzer
- added D12: EMERALD_LED, LED_SMD:LED_0402_1005Metric, symbol Device:LED_Small
- added D13: ORANGE_LED, LED_SMD:LED_0402_1005Metric, symbol Device:LED_Small
- added R38, R39: 470, Resistor_SMD:R_0402_1005Metric, symbol Device:R_Small
- added TP24: TestPoint, TestPoint:TestPoint_Pad_D1.0mm, symbol Connector:TestPoint
- U2: value DPS310 -> DPS368
Connections:
- net +3V3: now also BZ1.1 (+), R38.1, R39.1
- net CAN_RX: now also D13.1 (K)
- net CAN_TX: now also D12.1 (K)
- net at J2.1 (Pin_1), Q1.3 (D), R11.2: now also BZ1.2 (-)
- net DepVolt: now reaches U1.51 (GPIO45)
- new net: D12.2 (A), R38.2
- new net: D13.2 (A), R39.2
- new net PPS: TP24.1
- no-connect marks 14 -> 11
Other:
- sheet GPS ports: added PPS; removed none
- sheet power ports: added Dep_Volt_Scaled, Logic_Volt_Scaled; removed UC_Lipo_Scaled
- moved on the sheet: J2

Commit message: more hardware updates
Parts:
- removed 12VLED1: RED_LED, LED_SMD:LED_0402_1005Metric, symbol Device:LED_Small
- removed BZ1: CMT-0525-75-SMT-TR, symbol Device:Buzzer
- removed C12: DNP, Capacitor_SMD:C_0402_1005Metric, symbol Device:C_Small
- removed J3: 292227-7, iclr:292227-7, symbol iclr:292227-7
- removed J4: Micro_SD_Card_Det, Connector_Card:microSD_HC_Hirose_DM3AT-SF-PEJM5, symbol Connector:Micro_SD_Card_Det_Hirose_DM3AT
- removed R10: 5.1k, Resistor_SMD:R_0402_1005Metric, symbol Device:R_Small
- removed R12: 10k, Resistor_SMD:R_0402_1005Metric, symbol Device:R_Small
- removed TP1, TP12, TP14, TP18, TP19, TP2, TP20, TP21, TP3, TP4: TestPoint, TestPoint:TestPoint_Pad_D1.0mm, symbol Connector:TestPoint
- added J14: Conn_01x07_Socket, Connector_Molex:Molex_Pico-Clasp_202396-0707_1x07-1MP_P1.00mm_Horizontal, symbol Connector:Conn_01x07_Socket
- added J3: ST1W008S4TR2000, iclr-hw:JAE_ST1W008S4TR2000, symbol iclr-hw:ST1W008S4TR2000
- added LS1: CMT-0525-75-SMT-TR, iclr-hw:CMT052575SMTTR, symbol iclr-hw:CMT-0525-75-SMT-TR
- added R48: 10k, Resistor_SMD:R_0402_1005Metric, symbol Device:R_Small
- R8: value DNP -> 0
Connections:
- net BattVolt is gone; now on net LogicVolt: U1.7 (GPIO2/ADC1_CH1)
- net +3V3: now also J14.7 (Pin_7), J3.C4, LS1.1 (+), R48.1
- net DepVolt: now also U1.22 (GPIO16/ADC2_CH5/XTAL_32K_N); no longer U1.51 (GPIO45)
- net GND: now also J14.4 (Pin_4), J3.C6, J3.GND1 (GND), J3.GND2 (GND), J3.GND3 (GND), J3.GND4 (GND); no longer R8.1
- net JTAG_MTCK: now also R8.2
- net PPS: now also R8.1
- net SD1_CS: now also J3.C2
- net SD1_DET: now also J3.SW, R48.2
- net SD2_CS: now also J14.2 (Pin_2)
- net SD2_DET: now also J14.1 (Pin_1)
- net VSPI_MISO: now also J14.6 (Pin_6), J3.C7
- net VSPI_MOSI: now also J14.3 (Pin_3), J3.C3
- net VSPI_SCLK: now also J14.5 (Pin_5), J3.C5
- net at J2.1 (Pin_1), Q1.3 (D), R11.2: now also LS1.2 (-)
- net DepCurrent: now reaches U1.21 (GPIO15/ADC2_CH4/XTAL_32K_P)
- net ABUS_RX: now reaches U1.36 (SPICLK_N/GPIO48)
- net ABUS_TX: now reaches U1.37 (SPICLK_P/GPIO47)
- no-connect marks 11 -> 14
Other:
- added sheet ABUS (abus.kicad_sch)
- sheet power ports: added DepCurrent, EFuse_PG; removed none
- moved on the sheet: C13, C14, TP24, TP5, TP6, Y1

Commit message: progress
Parts:
- added J4: Conn_01x03_Pin, Connector_PinHeader_2.54mm:PinHeader_1x03_P2.54mm_Vertical, symbol Connector:Conn_01x03_Pin
Connections:
- net JTAG_MTDI: now also J4.2 (Pin_2)
- net JTAG_MTDO: now also J4.1 (Pin_1)
- net JTAG_MTMS: now also J4.3 (Pin_3)
- net LORA_INT: now also U1.9 (GPIO4/ADC1_CH3); no longer U1.10 (GPIO5/ADC1_CH4)
- net SD1_CS: now also U1.13 (GPIO8/ADC1_CH7); no longer U1.9 (GPIO4/ADC1_CH3)
- net SD1_DET: now also U1.10 (GPIO5/ADC1_CH4); no longer U1.11 (GPIO6/ADC1_CH5)
- net SD2_CS: now also U1.12 (GPIO7/ADC1_CH6); no longer U1.13 (GPIO8/ADC1_CH7)
- net SD2_DET: now also U1.11 (GPIO6/ADC1_CH5); no longer U1.12 (GPIO7/ADC1_CH6)
Other:
- moved on the sheet: C1, C5
