File: Hardware/PickleRick.kicad_sch (KiCad schematic)
At the start: 64 parts, among them J101 Conn_01x02_Male, J102 Conn_01x03_Pin, J103 Conn_01x02_Male, J104 Conn_02x03_Pin, J105 Conn_01x02_Male, J106 ST1W008S4TR2000, J107 Conn_01x07_Socket, J108 Conn_01x03_Male, Q101 PMV20ENR, U101 ESP32-S3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

Commit message: continued
Parts:
- D108: footprint iclr-hw:RCLAMP3346PQTNT -> iclr:RCLAMP3346PQTNT
- J106: footprint iclr-hw:JAE_ST1W008S4TR2000 -> iclr:JAE_ST1W008S4TR2000
- Y101: value 40MHz -> 40MHz±10ppm; footprint iclr:Crystal_SMD_2016-4Pin_2.0x1.6mm -> Crystal:Crystal_SMD_2016-4Pin_2.0x1.6mm
Changed lines of the file:
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@@
 			)
 		)
-		(property "Footprint" "iclr-hw:JAE_ST1W008S4TR2000"
+		(property "Footprint" "iclr:JAE_ST1W008S4TR2000"
 			(at 252.73 100.076 0)
 			(effects
@@
 			)
 		)
-		(property "Footprint" "iclr-hw:RCLAMP3346PQTNT"
+		(property "Footprint" "iclr:RCLAMP3346PQTNT"
 			(at 160.02 275.26 0)
 			(effects
@@
 			)
 		)
-		(property "Value" "40MHz"
+		(property "Value" "40MHz±10ppm"
 			(at 153.67 124.46 90)
 			(effects
@@
 			)
 		)
-		(property "Footprint" "iclr:Crystal_SMD_2016-4Pin_2.0x1.6mm"
+		(property "Footprint" "Crystal:Crystal_SMD_2016-4Pin_2.0x1.6mm"
 			(at 160.02 132.08 0)
 			(effects
