File: Hardware/PickleRick.kicad_pcb (KiCad board)
At the start: 4 copper layers, 100 x 37 mm, 205 parts, among them IC1 TPS259830ONRGER, J1 RBUS, J10 Conn_Coaxial, J11 Conn_Coaxial, J12 Conn_01x03_Male, J13 Conn_01x03_Pin, J14 Conn_01x07_Socket, J2 Conn_01x02_Male, J3 ST1W008S4TR2000, J4 Conn_01x03_Pin, J5 USB_C_Receptacle_USB2.0, J6 Screw_Terminal_01x08, J7 Conn_01x05_Male, J8 DeployLipo, J9 UCLipo, Q1 PMV20ENR, Q10 DMP3099L, Q11 SQS141ELNW-T1_GE3, Q12 SQS141ELNW-T1_GE3, Q2 BUK9M11-40EX, Q3 BUK9M11-40EX, Q4 BUK9M11-40EX, Q5 BUK9M11-40EX, Q8 DMP3099L, Q9 DMP3099L, U1 ESP32-S3, U10 LTC4412xS6, U11 MP28167GQ-A-Z, U14 LTC4412xS6, U16 SC4215, U17 LTC4412xS6, U19 MAX-M10S, U2 DPS368, U20 SN65HVD230, U21 RFM95W-868S2, U22 LTC4412xS6, U3 LTV-247, U4 PCA9534RGVR, U5 PCA9685BS, U6 H3LIS331DLTR, U7 ICM-20608-G, U8 MMC5983MA, U9 LTC4412xS6, Y1 R940000171

Commit message: hardware update
Parts:
- added D19: RCLAMP3346PQTNT, iclr-hw:RCLAMP3346PQTNT, F.Cu at (181.4, 89.2)
- moved R8 0.60 mm to (120.6, 78.4)
- moved C10 0.30 mm to (178.3, 87.8)
Routing:
- net GND: track 110.5 -> 113.0 mm, vias 230 -> 231
- net /JTAG_MTCK: track 86.4 -> 84.8 mm
- net +3V3: track 70.4 -> 71.2 mm
- net /DepCurrent: track 71.3 -> 70.8 mm

Commit message: update
Parts:
- R47: value 681 -> 680
- moved G*** 6.98 mm to (131.5, 74.2)
- moved G*** 4.61 mm to (125.1, 74.3)
- moved TP24 0.17 mm to (122.7, 67.4)
- moved TP5 0.15 mm to (122.7, 69.4)
- moved TP25 0.11 mm to (158.7, 84.2)
- moved C7 0.10 mm to (175.0, 79.4)
- moved TP6 0.10 mm to (122.7, 71.4)
- moved C27 0.07 mm to (148.6, 78.7)
- moved TP22 0.07 mm to (153.5, 94.5)
- moved R6 0.06 mm to (186.2, 91.8)
- moved TP23 0.06 mm to (153.4, 92.5)
- moved J2 0.06 mm to (191.5, 63.3)
- moved L1 0.06 mm to (174.6, 80.8)
- moved TP16 0.06 mm to (181.5, 74.8)
- moved Q11 0.05 mm to (153.4, 74.6)
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Routing:
- net +3V3: track 71.2 -> 79.2 mm

Commit message: more updates to hardware
Parts:
- moved G*** 1.66 mm to (133.1, 74.2)
- moved G*** 1.28 mm to (126.3, 74.0)
Routing:
- net /SCL: track 142.2 -> 142.8 mm
- net /JTAG_MTDO: track 10.7 -> 10.1 mm
- net /MAG_CS: track 33.0 -> 32.5 mm
- net GND: track 112.9 -> 112.4 mm

Commit message: update
Routing:
- net /SCL: track 142.8 -> 144.0 mm
