File: Hardware/power.kicad_sch (KiCad schematic)
At the start: 71 parts, among them IC1 MIC5060YML-TR, J8 DeployLipo, J9 UCLipo, Q10 DMP3099L, Q11 SQS141ELNW-T1_GE3, Q12 SQS141ELNW-T1_GE3, Q5 BSZ025N04LS, Q8 DMP3099L, Q9 DMP3099L, U10 LTC4412xS6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

Commit message: Updated Baseboard design but with power supply problems
Parts:
- renumbered 12VLED1 to 12VLED501, C29 to C501, C35 to C502, C31 to C503, C37 to C504, C38 to C505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
