File: Hardware/Nukes.kicad_sch (KiCad schematic)
At the start: 41 parts, among them J6 Screw_Terminal_01x08, J7 Conn_01x05_Male, Q2 BSZ025N04LS, Q3 BSZ025N04LS, Q4 BSZ025N04LS, Q6 BSZ025N04LS, U3 LTV-247, U4 PCA9534RGVR, U5 PCA9685BS

Commit message: cleaned up schematic and bom
Parts:
- D901: renamed from D20; value EMERALD_LED -> LED_GREEN
- D902: renamed from D21; value EMERALD_LED -> LED_GREEN
- D903: renamed from D8; value D_Schottky -> DST1550S
- D904: renamed from D7; value D_Schottky -> DST1550S
- D905: renamed from D27; value RED_LED -> LED_RED
- D906: renamed from D26; value RED_LED -> LED_RED
- D909: renamed from D22; value EMERALD_LED -> LED_GREEN
- D910: renamed from D9; value D_Schottky -> DST1550S
- D911: renamed from D25; value RED_LED -> LED_RED
- D913: renamed from D23; value EMERALD_LED -> LED_GREEN
- D914: renamed from D10; value D_Schottky -> DST1550S
- D915: renamed from D24; value RED_LED -> LED_RED
- R901: renamed from R12; value 120 -> 120Ω
- R902: renamed from R49; value 120 -> 120Ω
- R903: renamed from R18; value 120 -> 120Ω
- R904: renamed from R17; value 120 -> 120Ω
- R905: renamed from R50; value 120 -> 120Ω
- R906: renamed from R21; value 120 -> 120Ω
- R907: renamed from R51; value 120 -> 120Ω
- R908: renamed from R22; value 120 -> 120Ω
- R909: renamed from R47; value 220 -> 220Ω
- R910: renamed from R52; value 220 -> 220Ω
- R911: renamed from R53; value 220 -> 220Ω
- R912: renamed from R54; value 220 -> 220Ω
- renumbered C17 to C901, C18 to C902, C19 to C903, C20 to C904, D14 to D907, D17 to D908, D16 to D912, D15 to D916, J6 to J901, J7 to J902, Q2 to Q901, Q3 to Q902, Q6 to Q903, Q4 to Q904, U3 to U901, U4 to U902, U5 to U903
