File: Hardware/usb-uart.kicad_sch (KiCad schematic)
At the start: 9 parts, among them J5 USB_C_Receptacle_USB2.0

Commit message: black edition ordering stuff
Parts:
- R16: value 470 -> 5k
- USBLED1: value USB_LED -> WHITE_LED; footprint Resistor_SMD:R_0402_1005Metric -> LED_SMD:LED_0402_1005Metric
Changed lines of the file:
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@@
       (effects (font (size 1.27 1.27)))
     )
-    (property "Value" "USB_LED" (at 162.56 89.8144 0)
+    (property "Value" "WHITE_LED" (at 162.56 89.8144 0)
       (effects (font (size 1.27 1.27)))
     )
-    (property "Footprint" "Resistor_SMD:R_0402_1005Metric" (at 162.56 92.71 90)
+    (property "Footprint" "LED_SMD:LED_0402_1005Metric" (at 162.56 92.71 90)
       (effects (font (size 1.27 1.27)) hide)
     )
@@
       (effects (font (size 1.27 1.27)))
     )
-    (property "Value" "470" (at 154.94 95.377 90)
+    (property "Value" "5k" (at 154.94 95.377 90)
       (effects (font (size 1.27 1.27)))
     )

Commit message: fixes
Parts:
- R16: value 5k -> 5.1k
Changed lines of the file:
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@@
 			)
 		)
-		(property "Value" "5k"
+		(property "Value" "5.1k"
 			(at 154.94 95.377 90)
 			(effects

Commit message: Adding some 3d models
Parts:
- J5: footprint Connector_USB:USB_C_Receptacle_Palconn_UTC16-G -> iclr:USB_C_Receptacle_Palconn_UTC16-G
Changed lines of the file:
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@@
 	(label "Data+"
 		(at 132.08 134.62 90)
-		(fields_autoplaced yes)
 		(effects
 			(font
@@
 	(label "VBUS"
 		(at 129.54 134.62 90)
-		(fields_autoplaced yes)
 		(effects
 			(font
@@
 	(label "Data+"
 		(at 44.45 104.14 0)
-		(fields_autoplaced yes)
 		(effects
 			(font
@@
 	(label "Data-"
 		(at 44.45 99.06 0)
-		(fields_autoplaced yes)
 		(effects
 			(font
@@
 	(label "Data-"
 		(at 134.62 134.62 90)
-		(fields_autoplaced yes)
 		(effects
 			(font
@@
 	(label "Data-"
 		(at 116.84 102.87 0)
-		(fields_autoplaced yes)
 		(effects
 			(font
@@
 	(label "VBUS"
 		(at 44.45 109.22 0)
-		(fields_autoplaced yes)
 		(effects
 			(font
@@
 	(label "Data+"
 		(at 116.84 107.95 0)
-		(fields_autoplaced yes)
 		(effects
 			(font
@@
 		(shape bidirectional)
 		(at 44.45 99.06 180)
-		(fields_autoplaced yes)
 		(effects
 			(font
@@
 		(shape bidirectional)
 		(at 44.45 104.14 180)
-		(fields_autoplaced yes)
 		(effects
 			(font
@@
 			)
 		)
-		(property "Footprint" "Connector_USB:USB_C_Receptacle_Palconn_UTC16-G"
+		(property "Footprint" "iclr:USB_C_Receptacle_Palconn_UTC16-G"
 			(at 104.14 104.14 0)
 			(effects

Commit message: cleaned up schematic and bom
Parts:
- D802: renamed from USBLED1; value WHITE_LED -> LED_WHITE
- R801: renamed from R14; value 5.1k -> 5.1kΩ
- R802: renamed from R15; value 5.1k -> 5.1kΩ
- R803: renamed from R16; value 5.1k -> 5.1kΩ
- TP801: renamed from TP7; now left out of the parts list
- TP802: renamed from TP8; now left out of the parts list
- TP803: renamed from TP9; now left out of the parts list
- renumbered D6 to D801, J5 to J801
Changed lines of the file:
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@@
 (kicad_sch
-	(version 20231120)
+	(version 20250114)
 	(generator "eeschema")
-	(generator_version "8.0")
+	(generator_version "9.0")
 	(paper "A4")
 	(junction
@@
 	(wire
 		(pts
+			(xy 149.86 92.71) (xy 152.4 92.71)
+		)
+		(stroke
+			(width 0)
+			(type default)
+		)
+	)
+	(wire
+		(pts
 			(xy 160.02 92.71) (xy 157.48 92.71)
 		)
@@
 	(wire
 		(pts
+			(xy 167.64 92.71) (xy 165.1 92.71)
+		)
+		(stroke
+			(width 0)
+			(type default)
+		)
+	)
+	(wire
+		(pts
 			(xy 125.73 93.98) (xy 125.73 96.52)
 		)
@@
 	(wire
 		(pts
-			(xy 125.73 96.52) (xy 127 96.52)
+			(xy 125.73 96.52) (xy 130.81 96.52)
 		)
 		(stroke
@@
 	(symbol
 		(lib_id "power:GND")
-		(at 127 96.52 90)
+		(at 130.81 96.52 0)
 		(unit 1)
 		(exclude_from_sim no)
@@
 		(on_board yes)
 		(dnp no)
-		(property "Reference" "#PWR038"
-			(at 133.35 96.52 0)
+		(property "Reference" "#PWR0803"
+			(at 130.81 102.87 0)
 			(effects
 				(font
@@
 		)
 		(property "Value" "GND"
-			(at 130.2512 96.393 90)
+			(at 134.112 100.076 0)
 			(effects
 				(font
@@
 		)
 		(property "Footprint" ""
-			(at 127 96.52 0)
+			(at 130.81 96.52 0)
 			(effects
 				(font
@@
 		)
 		(property "Datasheet" ""
-			(at 127 96.52 0)
-			(effects
-				(font
-					(size 1.27 1.27)
-				)
-				(hide yes)
-			)
-		)
-		(property "Description" ""
-			(at 127 96.52 0)
+			(at 130.81 96.52 0)
+			(effects
+				(font
+					(size 1.27 1.27)
+				)
+				(hide yes)
+			)
+		)
+		(property "Description" ""
+			(at 130.81 96.52 0)
 			(effects
 				(font
@@
 			(project "PickleRick"
 				(path "/e63e39d7-6ac0-4ffd-8aa3-1841a4541b55/dd5f5a5e-a654-455b-bff7-78de55e53413"
-					(reference "#PWR038")
+					(reference "#PWR0803")
 					(unit 1)
 				)
@@
 		(on_board yes)
 		(dnp no)
-		(property "Reference" "R15"
-			(at 129.54 100.33 90)
-			(effects
-				(font
-					(size 1.27 1.27)
-				)
-			)
-		)
-		(property "Value" "5.1k"
-			(at 129.54 102.6414 90)
+		(property "Reference" "R802"
+			(at 126.492 101.3206 90)
+			(effects
+				(font
+					(size 1.27 1.27)
+				)
+			)
+		)
+		(property "Value" "5.1kΩ"
+			(at 126.492 103.632 90)
 			(effects
 				(font
@@
 			(project "PickleRick"
 				(path "/e63e39d7-6ac0-4ffd-8aa3-1841a4541b55/dd5f5a5e-a654-455b-bff7-78de55e53413"
-					(reference "R15")
+					(reference "R802")
 					(unit 1)
 				)
@@
 		(on_board yes)
 		(dnp no)
-		(property "Reference" "R14"
+		(property "Reference" "R801"
 			(at 123.19 89.0016 90)
 			(effects
@@
 			)
 		)
-		(property "Value" "5.1k"
+		(property "Value" "5.1kΩ"
 			(at 123.19 91.313 90)
 			(effects
@@
 			(project "PickleRick"
 				(path "/e63e39d7-6ac0-4ffd-8aa3-1841a4541b55/dd5f5a5e-a654-455b-bff7-78de55e53413"
-					(reference "R14")
+					(reference "R801")
 					(unit 1)
 				)
@@
 		(on_board yes)
 		(dnp no)
-		(property "Reference" "#PWR036"
+		(property "Reference" "#PWR0801"
 			(at 96.52 137.16 0)
 			(effects
@@
 			(project "PickleRick"
 				(path "/e63e39d7-6ac0-4ffd-8aa3-1841a4541b55/dd5f5a5e-a654-455b-bff7-78de55e53413"
-					(reference "#PWR036")
+					(reference "#PWR0801")
 					(unit 1)
 				)
@@
 		(on_board yes)
 		(dnp no)
-		(property "Reference" "J5"
+		(property "Reference" "J801"
 			(at 103.0478 82.1182 0)
 			(effects
@@
 			(project "PickleRick"
 				(path "/e63e39d7-6ac0-4ffd-8aa3-1841a4541b55/dd5f5a5e-a654-455b-bff7-78de55e53413"
-					(reference "J5")
+					(reference "J801")
 					(unit 1)
 				)
@@
 		(on_board yes)
 		(dnp no)
-		(property "Reference" "#PWR039"
+		(property "Reference" "#PWR0804"
 			(at 132.08 151.13 0)
 			(effects
@@
 			(project "PickleRick"
 				(path "/e63e39d7-6ac0-4ffd-8aa3-1841a4541b55/dd5f5a5e-a654-455b-bff7-78de55e53413"
-					(reference "#PWR039")
+					(reference "#PWR0804")
 					(unit 1)
 				)
@@
 		(on_board yes)
 		(dnp no)
-		(property "Reference" "D6"
+		(property "Reference" "D801"
 			(at 137.287 138.5316 0)
 			(effects
@@
 			(project "PickleRick"
 				(path "/e63e39d7-6ac0-4ffd-8aa3-1841a4541b55/dd5f5a5e-a654-455b-bff7-78de55e53413"
-					(reference "D6")
+					(reference "D801")
 					(unit 1)
 				)
@@
 		(on_board yes)
 		(dnp no)
-		(property "Reference" "#PWR037"
+		(property "Reference" "#PWR0802"
 			(at 116.84 88.9 0)
 			(effects
@@
 			(project "PickleRick"
 				(path "/e63e39d7-6ac0-4ffd-8aa3-1841a4541b55/dd5f5a5e-a654-455b-bff7-78de55e53413"
-					(reference "#PWR037")
+					(reference "#PWR0802")
 					(unit 1)
 				)
@@
 		(unit 1)
 		(exclude_from_sim no)
-		(in_bom yes)
-		(on_board yes)
-		(dnp no)
-		(property "Reference" "TP7"
+		(in_bom no)
+		(on_board yes)
+		(dnp no)
+		(property "Reference" "TP801"
 			(at 56.8452 97.8916 90)
 			(effects
@@
 			(project "PickleRick"
 				(path "/e63e39d7-6ac0-4ffd-8aa3-1841a4541b55/dd5f5a5e-a654-455b-bff7-78de55e53413"
-					(reference "TP7")
+					(reference "TP801")
 					(unit 1)
 				)
@@
 		(unit 1)
 		(exclude_from_sim no)
-		(in_bom yes)
-		(on_board yes)
-		(dnp no)
-		(property "Reference" "TP8"
+		(in_bom no)
+		(on_board yes)
+		(dnp no)
+		(property "Reference" "TP802"
 			(at 56.8452 102.9716 90)
 			(effects
@@
 			(project "PickleRick"
 				(path "/e63e39d7-6ac0-4ffd-8aa3-1841a4541b55/dd5f5a5e-a654-455b-bff7-78de55e53413"
-					(reference "TP8")
+					(reference "TP802")
 					(unit 1)
 				)
@@
 		(unit 1)
 		(exclude_from_sim no)
-		(in_bom yes)
-		(on_board yes)
-		(dnp no)
-		(property "Reference" "TP9"
+		(in_bom no)
+		(on_board yes)
+		(dnp no)
+		(property "Reference" "TP803"
 			(at 56.8452 108.0516 90)
 			(effects
@@
 			(project "PickleRick"
 				(path "/e63e39d7-6ac0-4ffd-8aa3-1841a4541b55/dd5f5a5e-a654-455b-bff7-78de55e53413"
-					(reference "TP9")
+					(reference "TP803")
 					(unit 1)
 				)
@@
 		(on_board yes)
 		(dnp no)
-		(property "Reference" "USBLED1"
+		(property "Reference" "D802"
 			(at 162.56 87.503 0)
 			(effects
@@
 			)
 		)
-		(property "Value" "WHITE_LED"
+		(property "Value" "LED_WHITE"
 			(at 162.56 89.8144 0)
 			(effects
@@
 			(project "PickleRick"
 				(path "/e63e39d7-6ac0-4ffd-8aa3-1841a4541b55/dd5f5a5e-a654-455b-bff7-78de55e53413"
-					(reference "USBLED1")
+					(reference "D802")
 					(unit 1)
 				)
@@
 		(on_board yes)
 		(dnp no)
-		(property "Reference" "R16"
+		(property "Reference" "R803"
 			(at 154.94 97.6884 90)
 			(effects
@@
 			)
 		)
-		(property "Value" "5.1k"
+		(property "Value" "5.1kΩ"
 			(at 154.94 95.377 90)
 			(effects
@@
 			(project "PickleRick"
 				(path "/e63e39d7-6ac0-4ffd-8aa3-1841a4541b55/dd5f5a5e-a654-455b-bff7-78de55e53413"
-					(reference "R16")
+					(reference "R803")
 					(unit 1)
 				)
@@
 	(symbol
 		(lib_id "power:GND")
-		(at 165.1 92.71 90)
+		(at 167.64 92.71 0)
 		(unit 1)
 		(exclude_from_sim no)
@@
 		(on_board yes)
 		(dnp no)
-		(property "Reference" "#PWR041"
-			(at 171.45 92.71 0)
+		(property "Reference" "#PWR0806"
+			(at 167.64 99.06 0)
 			(effects
 				(font
@@
 		)
 		(property "Value" "GND"
-			(at 168.3512 92.583 90)
+			(at 169.418 97.282 0)
 			(effects
 				(font
@@
 		)
 		(property "Footprint" ""
-			(at 165.1 92.71 0)
+			(at 167.64 92.71 0)
 			(effects
 				(font
@@
 		)
 		(property "Datasheet" ""
-			(at 165.1 92.71 0)
-			(effects
-				(font
-					(size 1.27 1.27)
-				)
-				(hide yes)
-			)
-		)
-		(property "Description" ""
-			(at 165.1 92.71 0)
+			(at 167.64 92.71 0)
+			(effects
+				(font
+					(size 1.27 1.27)
+				)
+				(hide yes)
+			)
+		)
+		(property "Description" ""
+			(at 167.64 92.71 0)
 			(effects
 				(font
@@
 			(project "PickleRick"
 				(path "/e63e39d7-6ac0-4ffd-8aa3-1841a4541b55/dd5f5a5e-a654-455b-bff7-78de55e53413"
-					(reference "#PWR041")
+					(reference "#PWR0806")
 					(unit 1)
 				)
@@
 	(symbol
 		(lib_id "power:VBUS")
-		(at 152.4 92.71 90)
+		(at 149.86 92.71 0)
 		(unit 1)
 		(exclude_from_sim no)
@@
 		(on_board yes)
 		(dnp no)
-		(property "Reference" "#PWR040"
-			(at 156.21 92.71 0)
+		(property "Reference" "#PWR0805"
+			(at 149.86 96.52 0)
 			(effects
 				(font
@@
 		)
 		(property "Value" "VBUS"
-			(at 149.1488 92.329 90)
+			(at 147.574 88.646 0)
 			(effects
 				(font
@@
 		)
 		(property "Footprint" ""
-			(at 152.4 92.71 0)
+			(at 149.86 92.71 0)
 			(effects
 				(font
@@
 		)
 		(property "Datasheet" ""
-			(at 152.4 92.71 0)
-			(effects
-				(font
-					(size 1.27 1.27)
-				)
-				(hide yes)
-			)
-		)
-		(property "Description" ""
-			(at 152.4 92.71 0)
+			(at 149.86 92.71 0)
+			(effects
+				(font
+					(size 1.27 1.27)
+				)
+				(hide yes)
+			)
+		)
+		(property "Description" ""
+			(at 149.86 92.71 0)
 			(effects
 				(font
@@
 			(project "PickleRick"
 				(path "/e63e39d7-6ac0-4ffd-8aa3-1841a4541b55/dd5f5a5e-a654-455b-bff7-78de55e53413"
-					(reference "#PWR040")
-					(unit 1)
-				)
+					(reference "#PWR0805")
+					(unit 1)
+				)
