File: Hardware/abus.kicad_sch (KiCad schematic)
At the start: 2 parts, among them J13 Conn_01x03_Pin

Commit message: progress
Connections:
- net RX: now also D18.5, J13.3 (Pin_3); no longer D18.1, J13.2 (Pin_2)
- net TX: now also D18.1, J13.2 (Pin_2); no longer D18.5, J13.3 (Pin_3)
Other:
- moved on the sheet: D18A
Changed lines of the file:
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@@
+	(wire
+		(pts
+			(xy 87.9356 73.835) (xy 87.9356 76.375)
+		)
+		(stroke
+			(width 0)
+			(type default)
+		)
+	)
 	(wire
 		(pts
@@
 	(hierarchical_label "TX"
 		(shape input)
+		(at 92.71 69.85 0)
+		(fields_autoplaced yes)
+		(effects
+			(font
+				(size 1.27 1.27)
+			)
+			(justify left)
+		)
+	)
+	(hierarchical_label "RX"
+		(shape input)
+		(at 82.55 69.85 180)
+		(fields_autoplaced yes)
+		(effects
+			(font
+				(size 1.27 1.27)
+			)
+			(justify right)
+		)
+	)
+	(hierarchical_label "RX"
+		(shape input)
 		(at 121.92 66.04 180)
 		(fields_autoplaced yes)
@@
 		)
 	)
-	(hierarchical_label "RX"
-		(shape input)
-		(at 92.4044 72.215 0)
-		(fields_autoplaced yes)
-		(effects
-			(font
-				(size 1.27 1.27)
-			)
-			(justify left)
-		)
-	)
 	(hierarchical_label "TX"
-		(shape input)
-		(at 82.2444 72.215 180)
-		(fields_autoplaced yes)
-		(effects
-			(font
-				(size 1.27 1.27)
-			)
-			(justify right)
-		)
-	)
-	(hierarchical_label "RX"
 		(shape input)
 		(at 121.92 68.58 180)
@@
 	(symbol
 		(lib_id "power:GND")
-		(at 87.63 76.2 0)
+		(at 87.9356 76.375 0)
 		(unit 1)
 		(exclude_from_sim no)
@@
 		(fields_autoplaced yes)
 		(property "Reference" "#PWR0106"
-			(at 87.63 82.55 0)
+			(at 87.9356 82.725 0)
 			(effects
 				(font
@@
 		)
 		(property "Value" "GND"
-			(at 87.63 81.28 0)
+			(at 87.9356 81.455 0)
 			(effects
 				(font
@@
 		)
 		(property "Footprint" ""
-			(at 87.63 76.2 0)
+			(at 87.9356 76.375 0)
 			(effects
 				(font
@@
 		)
 		(property "Datasheet" ""
-			(at 87.63 76.2 0)
+			(at 87.9356 76.375 0)
 			(effects
 				(font
@@
 		)
 		(property "Description" "Power symbol creates a global label with name \"GND\" , ground"
-			(at 87.63 76.2 0)
+			(at 87.9356 76.375 0)
 			(effects
 				(font
@@
 	(symbol
 		(lib_id "iclr-hw:CPDV5-3V3UP")
-		(at 102.5644 72.215 270)
+		(at 102.87 69.85 270)
 		(unit 1)
 		(exclude_from_sim no)
@@
 		(fields_autoplaced yes)
 		(property "Reference" "D18"
-			(at 87.5944 67.135 90)
+			(at 87.9 64.77 90)
 			(effects
 				(font
@@
 		)
 		(property "Value" "~"
-			(at 87.5944 69.675 90)
+			(at 87.9 67.31 90)
 			(effects
 				(font
@@
 		)
 		(property "Footprint" "Package_TO_SOT_SMD:SOT-353_SC-70-5"
-			(at 95.7144 72.215 0)
+			(at 96.02 69.85 0)
 			(effects
 				(font
@@
 		)
 		(property "Datasheet" "https://www.mouser.co.uk/datasheet/2/80/CPDV5_3V3UP_HF_RevB181493-2505215.pdf"
-			(at 95.7144 72.215 0)
+			(at 96.02 69.85 0)
 			(effects
 				(font
@@
 		)
 		(property "Description" "2 channel double backed zener TVS diode"
-			(at 95.7144 72.215 0)
-			(effects
-				(font
+			(at 96.02 69.85 0)
+			(effects
+				(font

Commit message: update
Parts:
- added unit 2 of D18
Connections:
- net GND: now also D18.1, D18.3; no longer D18.2
- net TX: now also D18.4; no longer D18.1
- new net: D18.2, D18.2
Changed lines of the file:
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@@
-	(wire
-		(pts
-			(xy 87.9356 73.835) (xy 87.9356 76.375)
-		)
-		(stroke
-			(width 0)
-			(type default)
-		)
-	)
 	(wire
 		(pts
@@
 	(wire
 		(pts
+			(xy 92.71 74.93) (xy 92.71 78.74)
+		)
+		(stroke
+			(width 0)
+			(type default)
+		)
+	)
+	(wire
+		(pts
 			(xy 119.38 71.12) (xy 119.38 74.93)
 		)
@@
 		)
 	)
-	(hierarchical_label "TX"
+	(wire
+		(pts
+			(xy 100.33 74.93) (xy 100.33 80.01)
+		)
+		(stroke
+			(width 0)
+			(type default)
+		)
+	)
+	(hierarchical_label "RX"
 		(shape input)
-		(at 92.71 69.85 0)
+		(at 100.33 62.23 90)
 		(fields_autoplaced yes)
 		(effects
@@
 	(hierarchical_label "RX"
 		(shape input)
-		(at 82.55 69.85 180)
+		(at 121.92 66.04 180)
 		(fields_autoplaced yes)
 		(effects
@@
 		)
 	)
-	(hierarchical_label "RX"
+	(hierarchical_label "TX"
 		(shape input)
-		(at 121.92 66.04 180)
+		(at 92.71 62.23 90)
 		(fields_autoplaced yes)
 		(effects
@@
 				(size 1.27 1.27)
 			)
-			(justify right)
+			(justify left)
 		)
 	)
@@
 			)
 			(justify right)
+		)
+	)
+	(symbol
+		(lib_name "CPDV5-3V3UP_1")
+		(lib_id "iclr-hw:CPDV5-3V3UP")
+		(at 92.71 53.34 0)
+		(unit 2)
+		(exclude_from_sim no)
+		(in_bom yes)
+		(on_board yes)
+		(dnp no)
+		(fields_autoplaced yes)
+		(property "Reference" "D18"
+			(at 87.63 68.5851 90)
+			(effects
+				(font
+					(size 1.27 1.27)
+				)
+			)
+		)
+		(property "Value" "~"
+			(at 90.17 68.5851 90)
+			(effects
+				(font
+					(size 1.27 1.27)
+				)
+			)
+		)
+		(property "Footprint" "Package_TO_SOT_SMD:SOT-353_SC-70-5"
+			(at 92.71 60.19 0)
+			(effects
+				(font
+					(size 1.27 1.27)
+				)
+				(hide yes)
+			)
+		)
+		(property "Datasheet" "https://www.mouser.co.uk/datasheet/2/80/CPDV5_3V3UP_HF_RevB181493-2505215.pdf"
+			(at 92.71 60.19 0)
+			(effects
+				(font
+					(size 1.27 1.27)
+				)
+				(hide yes)
+			)
+		)
+		(property "Description" "2 channel double backed zener TVS diode"
+			(at 92.71 60.19 0)
+			(effects
+				(font
+					(size 1.27 1.27)
+				)
+				(hide yes)
+			)
+		)
+		(pin "1"
+		)
+		(pin "5"
+		)
+		(pin "2"
+		)
+		(pin "2"
+		)
+		(pin "4"
+		)
+		(pin "3"
+		)
+		(instances
+			(project ""
+				(path "/e63e39d7-6ac0-4ffd-8aa3-1841a4541b55/f8ca6ebe-a1b7-4d27-a7e8-9fa3d73c83bf"
+					(reference "D18")
+					(unit 2)
+				)
+			)
 		)
 	)
@@
 	)
 	(symbol
-		(lib_id "power:GND")
-		(at 87.9356 76.375 0)
+		(lib_id "iclr-hw:CPDV5-3V3UP")
+		(at 100.33 83.82 180)
 		(unit 1)
 		(exclude_from_sim no)
@@
 		(dnp no)
 		(fields_autoplaced yes)
-		(property "Reference" "#PWR0106"
-			(at 87.9356 82.725 0)
-			(effects
-				(font
-					(size 1.27 1.27)
-				)
-				(hide yes)
-			)
-		)
-		(property "Value" "GND"
-			(at 87.9356 81.455 0)
-			(effects
-				(font
-					(size 1.27 1.27)
-				)
-			)
-		)
-		(property "Footprint" ""
-			(at 87.9356 76.375 0)
-			(effects
-				(font
-					(size 1.27 1.27)
-				)
-				(hide yes)
-			)
-		)
-		(property "Datasheet" ""
-			(at 87.9356 76.375 0)
-			(effects
-				(font
-					(size 1.27 1.27)
-				)
-				(hide yes)
-			)
-		)
-		(property "Description" "Power symbol creates a global label with name \"GND\" , ground"
-			(at 87.9356 76.375 0)
-			(effects
-				(font
-					(size 1.27 1.27)
-				)
-				(hide yes)
-			)
+		(property "Reference" "D18"
+			(at 105.41 68.85 90)
+			(effects
+				(font
+					(size 1.27 1.27)
+				)
+			)
+		)
+		(property "Value" "~"
+			(at 102.87 68.85 90)
+			(effects
+				(font
+					(size 1.27 1.27)
+				)
+			)
+		)
+		(property "Footprint" "Package_TO_SOT_SMD:SOT-353_SC-70-5"
+			(at 100.33 76.97 0)
+			(effects
+				(font
+					(size 1.27 1.27)
+				)
+				(hide yes)
+			)
+		)
+		(property "Datasheet" "https://www.mouser.co.uk/datasheet/2/80/CPDV5_3V3UP_HF_RevB181493-2505215.pdf"
+			(at 100.33 76.97 0)
+			(effects
+				(font
+					(size 1.27 1.27)
+				)
+				(hide yes)
+			)
+		)
+		(property "Description" "2 channel double backed zener TVS diode"
+			(at 100.33 76.97 0)
+			(effects
+				(font
+					(size 1.27 1.27)
+				)
+				(hide yes)
+			)
+		)
+		(pin "4"
+		)
+		(pin "3"
+		)
+		(pin "5"
+		)
+		(pin "2"
 		)
 		(pin "1"
+		)
+		(pin "2"
 		)
 		(instances
 			(project ""
 				(path "/e63e39d7-6ac0-4ffd-8aa3-1841a4541b55/f8ca6ebe-a1b7-4d27-a7e8-9fa3d73c83bf"
-					(reference "#PWR0106")
+					(reference "D18")
 					(unit 1)
 				)
@@
 	)
 	(symbol
-		(lib_id "iclr-hw:CPDV5-3V3UP")
-		(at 102.87 69.85 270)
+		(lib_id "power:GND")
+		(at 92.71 78.74 0)
 		(unit 1)
 		(exclude_from_sim no)
@@
 		(dnp no)
 		(fields_autoplaced yes)
-		(property "Reference" "D18"
-			(at 87.9 64.77 90)
-			(effects
-				(font
-					(size 1.27 1.27)
-				)
-			)
-		)
-		(property "Value" "~"
-			(at 87.9 67.31 90)
-			(effects
-				(font
-					(size 1.27 1.27)
-				)
-			)
-		)
-		(property "Footprint" "Package_TO_SOT_SMD:SOT-353_SC-70-5"
-			(at 96.02 69.85 0)
-			(effects
-				(font
-					(size 1.27 1.27)
-				)
-				(hide yes)
-			)
-		)
-		(property "Datasheet" "https://www.mouser.co.uk/datasheet/2/80/CPDV5_3V3UP_HF_RevB181493-2505215.pdf"
-			(at 96.02 69.85 0)
-			(effects
-				(font
-					(size 1.27 1.27)
-				)
-				(hide yes)
-			)
-		)
-		(property "Description" "2 channel double backed zener TVS diode"
-			(at 96.02 69.85 0)
-			(effects
-				(font
-					(size 1.27 1.27)
-				)
-				(hide yes)
-			)
-		)
-		(pin "4"
-		)
-		(pin "3"
-		)
-		(pin "5"
-		)
-		(pin "2"
+		(property "Reference" "#PWR016"
+			(at 92.71 85.09 0)
+			(effects
+				(font
+					(size 1.27 1.27)
+				)
+				(hide yes)
+			)
+		)
+		(property "Value" "GND"
+			(at 92.71 83.82 0)
+			(effects
+				(font
+					(size 1.27 1.27)
+				)
+			)
+		)
+		(property "Footprint" ""
+			(at 92.71 78.74 0)
+			(effects
+				(font
+					(size 1.27 1.27)
+				)
+				(hide yes)
+			)
+		)
+		(property "Datasheet" ""
+			(at 92.71 78.74 0)
+			(effects
+				(font
+					(size 1.27 1.27)
+				)
+				(hide yes)
+			)
+		)
+		(property "Description" "Power symbol creates a global label with name \"GND\" , ground"
+			(at 92.71 78.74 0)
+			(effects
+				(font
+					(size 1.27 1.27)
+				)
+				(hide yes)
+			)
 		)
 		(pin "1"
-		)
-		(pin "2"
 		)
 		(instances
 			(project ""
 				(path "/e63e39d7-6ac0-4ffd-8aa3-1841a4541b55/f8ca6ebe-a1b7-4d27-a7e8-9fa3d73c83bf"
-					(reference "D18")
+					(reference "#PWR016")
 					(unit 1)
 				)
+			)
+		)
+	)
+	(symbol
+		(lib_id "power:GND")
+		(at 100.33 80.01 0)
+		(unit 1)
+		(exclude_from_sim no)
+		(in_bom yes)
+		(on_board yes)
+		(dnp no)
+		(fields_autoplaced yes)
+		(property "Reference" "#PWR0106"
+			(at 100.33 86.36 0)
+			(effects
+				(font
+					(size 1.27 1.27)
+				)
+				(hide yes)
+			)
+		)
+		(property "Value" "GND"
+			(at 100.33 85.09 0)
+			(effects
+				(font
+					(size 1.27 1.27)
+				)
+			)
+		)
+		(property "Footprint" ""
+			(at 100.33 80.01 0)
+			(effects
+				(font
+					(size 1.27 1.27)
+				)
+				(hide yes)
+			)
+		)
+		(property "Datasheet" ""
+			(at 100.33 80.01 0)
+			(effects
+				(font
+					(size 1.27 1.27)
+				)
+				(hide yes)
+			)
+		)
+		(property "Description" "Power symbol creates a global label with name \"GND\" , ground"
+			(at 100.33 80.01 0)
+			(effects
+				(font
+					(size 1.27 1.27)
+				)
+				(hide yes)
+			)
+		)
+		(pin "1"
+		)
+		(instances
+			(project "PickleRick"
+				(path "/e63e39d7-6ac0-4ffd-8aa3-1841a4541b55/f8ca6ebe-a1b7-4d27-a7e8-9fa3d73c83bf"
+					(reference "#PWR0106")
+					(unit 1)
+				)

Commit message: cleaned up schematic and bom
Parts:
- D501: renamed from D18; value ~ -> CPDV5-3V3UP
- renumbered J13 to J501
Changed lines of the file:
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@@
 (kicad_sch
-	(version 20231120)
+	(version 20250114)
 	(generator "eeschema")
-	(generator_version "8.0")
+	(generator_version "9.0")
 	(paper "A4")
 	(wire
@@
 		(dnp no)
 		(fields_autoplaced yes)
-		(property "Reference" "D18"
+		(property "Reference" "D501"
 			(at 87.63 68.5851 90)
 			(effects
@@
 			)
 		)
-		(property "Value" "~"
+		(property "Value" "CPDV5-3V3UP"
 			(at 90.17 68.5851 90)
 			(effects
@@
 		)
 		(instances
-			(project ""
+			(project "PickleRick"
 				(path "/e63e39d7-6ac0-4ffd-8aa3-1841a4541b55/f8ca6ebe-a1b7-4d27-a7e8-9fa3d73c83bf"
-					(reference "D18")
+					(reference "D501")
 					(unit 2)
 				)
@@
 		(dnp no)
 		(fields_autoplaced yes)
-		(property "Reference" "#PWR011"
+		(property "Reference" "#PWR0503"
 			(at 119.38 81.28 0)
 			(effects
@@
 		)
 		(instances
-			(project ""
+			(project "PickleRick"
 				(path "/e63e39d7-6ac0-4ffd-8aa3-1841a4541b55/f8ca6ebe-a1b7-4d27-a7e8-9fa3d73c83bf"
-					(reference "#PWR011")
+					(reference "#PWR0503")
 					(unit 1)
 				)
@@
 		(dnp no)
 		(fields_autoplaced yes)
-		(property "Reference" "D18"
+		(property "Reference" "D501"
 			(at 105.41 68.85 90)
 			(effects
@@
 			)
 		)
-		(property "Value" "~"
+		(property "Value" "CPDV5-3V3UP"
 			(at 102.87 68.85 90)
 			(effects
@@
 		)
 		(instances
-			(project ""
+			(project "PickleRick"
 				(path "/e63e39d7-6ac0-4ffd-8aa3-1841a4541b55/f8ca6ebe-a1b7-4d27-a7e8-9fa3d73c83bf"
-					(reference "D18")
+					(reference "D501")
 					(unit 1)
 				)
@@
 		(dnp no)
 		(fields_autoplaced yes)
-		(property "Reference" "#PWR016"
+		(property "Reference" "#PWR0501"
 			(at 92.71 85.09 0)
 			(effects
@@
 		)
 		(instances
-			(project ""
+			(project "PickleRick"
 				(path "/e63e39d7-6ac0-4ffd-8aa3-1841a4541b55/f8ca6ebe-a1b7-4d27-a7e8-9fa3d73c83bf"
-					(reference "#PWR016")
+					(reference "#PWR0501")
 					(unit 1)
 				)
@@
 		(dnp no)
 		(fields_autoplaced yes)
-		(property "Reference" "#PWR0106"
+		(property "Reference" "#PWR0502"
 			(at 100.33 86.36 0)
 			(effects
@@
 			(project "PickleRick"
 				(path "/e63e39d7-6ac0-4ffd-8aa3-1841a4541b55/f8ca6ebe-a1b7-4d27-a7e8-9fa3d73c83bf"
-					(reference "#PWR0106")
+					(reference "#PWR0502")
 					(unit 1)
 				)
@@
 		(dnp no)
 		(fields_autoplaced yes)
-		(property "Reference" "J13"
+		(property "Reference" "J501"
 			(at 130.81 67.3099 0)
 			(effects
@@
 		)
 		(instances
-			(project ""
+			(project "PickleRick"
 				(path "/e63e39d7-6ac0-4ffd-8aa3-1841a4541b55/f8ca6ebe-a1b7-4d27-a7e8-9fa3d73c83bf"
-					(reference "J13")
+					(reference "J501")
 					(unit 1)
 				)

Commit message: updated resistors w cap footprints
Parts:
- D501: value CPDV5-3V3UP -> CPDV5-3V3UP-HF
Changed lines of the file:
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@@
 		(fields_autoplaced yes)
 		(property "Reference" "D501"
-			(at 87.63 68.5851 90)
+			(at 90.17 67.3149 0)
 			(effects
 				(font
 					(size 1.27 1.27)
 				)
+				(justify right)
 			)
 		)
-		(property "Value" "CPDV5-3V3UP"
-			(at 90.17 68.5851 90)
+		(property "Value" "CPDV5-3V3UP-HF"
+			(at 90.17 69.8549 0)
 			(effects
 				(font
 					(size 1.27 1.27)
 				)
+				(justify right)
 			)
 		)
@@
 			)
 		)
-		(property "Value" "CPDV5-3V3UP"
+		(property "Value" "CPDV5-3V3UP-HF"
 			(at 102.87 68.85 90)
 			(effects
